File: keyboard.kicad_sch (KiCad schematic)
At the start: 6 parts, among them J6 Side keys, J7 Keyboard, Q3 BSS138

Commit message: WIP SOM update
Parts:
- renumbered R27 to R31, R28 to R32, R29 to R33
Changed lines of the file:
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@@
 	(title_block
 		(title "LinHT - Linux-based SDR handheld transceiver")
-		(date "5 June 2025")
+		(date "6 July 2025")
 		(rev "A")
 		(company "M17 Foundation")
-		(comment 1 "Author: Wojciech SP5WWP")
+		(comment 1 "Author: Wojciech SP5WWP, Andy OE3ANC")
 	)
 	(bus_alias "KBD"
@@
 		(dnp no)
 		(fields_autoplaced yes)
-		(property "Reference" "#PWR093"
+		(property "Reference" "#PWR071"
 			(at 130.81 121.92 0)
 			(effects
@@
 			(project ""
 				(path "/73efc1fc-21f6-4aef-9f73-508fe18fa32e/058c0cc5-75b0-4494-8e78-217aac2f1bdc"
-					(reference "#PWR093")
+					(reference "#PWR071")
 					(unit 1)
 				)
@@
 		(dnp no)
 		(fields_autoplaced yes)
-		(property "Reference" "R28"
+		(property "Reference" "R32"
 			(at 163.322 100.3878 0)
 			(effects
@@
 			(project "linht-hw"
 				(path "/73efc1fc-21f6-4aef-9f73-508fe18fa32e/058c0cc5-75b0-4494-8e78-217aac2f1bdc"
-					(reference "R28")
+					(reference "R32")
 					(unit 1)
 				)
@@
 		(dnp no)
 		(fields_autoplaced yes)
-		(property "Reference" "#PWR095"
+		(property "Reference" "#PWR073"
 			(at 165.1 113.03 0)
 			(effects
@@
 			(project "linht-hw"
 				(path "/73efc1fc-21f6-4aef-9f73-508fe18fa32e/058c0cc5-75b0-4494-8e78-217aac2f1bdc"
-					(reference "#PWR095")
+					(reference "#PWR073")
 					(unit 1)
 				)
@@
 		(dnp no)
 		(fields_autoplaced yes)
-		(property "Reference" "R27"
+		(property "Reference" "R31"
 			(at 156.718 82.6078 0)
 			(effects
@@
 			(project ""
 				(path "/73efc1fc-21f6-4aef-9f73-508fe18fa32e/058c0cc5-75b0-4494-8e78-217aac2f1bdc"
-					(reference "R27")
+					(reference "R31")
 					(unit 1)
 				)
@@
 		(dnp no)
 		(fields_autoplaced yes)
-		(property "Reference" "#PWR094"
+		(property "Reference" "#PWR072"
 			(at 154.94 113.03 0)
 			(effects
@@
 			(project "linht-hw"
 				(path "/73efc1fc-21f6-4aef-9f73-508fe18fa32e/058c0cc5-75b0-4494-8e78-217aac2f1bdc"
-					(reference "#PWR094")
+					(reference "#PWR072")
 					(unit 1)
 				)
@@
 		(dnp no)
 		(fields_autoplaced yes)
-		(property "Reference" "R29"
+		(property "Reference" "R33"
 			(at 171.45 90.0895 90)
 			(effects
@@
 			(project "linht-hw"
 				(path "/73efc1fc-21f6-4aef-9f73-508fe18fa32e/058c0cc5-75b0-4494-8e78-217aac2f1bdc"
-					(reference "R29")
+					(reference "R33")
 					(unit 1)
 				)
@@
 		(dnp no)
 		(fields_autoplaced yes)
-		(property "Reference" "#PWR092"
+		(property "Reference" "#PWR070"
 			(at 130.81 76.2 0)
 			(effects
@@
 			(project ""
 				(path "/73efc1fc-21f6-4aef-9f73-508fe18fa32e/058c0cc5-75b0-4494-8e78-217aac2f1bdc"
-					(reference "#PWR092")
+					(reference "#PWR070")
 					(unit 1)
 				)

Commit message: routed some signals
Other:
- moved on the sheet: J6
Changed lines of the file:
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@@
+		)
+	)
+	(hierarchical_label "SIDE_PTT"
+		(shape output)
+		(at 68.58 87.63 0)
+		(effects
+			(font
+				(size 1.27 1.27)
+			)
+			(justify left)
 		)
 	)
@@
 		)
 	)
+	(hierarchical_label "SIDE_BTN"
+		(shape output)
+		(at 68.58 91.44 0)
+		(effects
+			(font
+				(size 1.27 1.27)
+			)
+			(justify left)
+		)
+	)
 	(hierarchical_label "KBD"
 		(shape bidirectional)
@@
 	(symbol
 		(lib_id "Connector_Generic:Conn_01x05")
-		(at 41.91 74.93 0)
+		(at 55.88 85.09 0)
 		(mirror y)
 		(unit 1)
@@
 		(dnp no)
 		(property "Reference" "J6"
-			(at 39.878 73.7178 0)
+			(at 53.848 83.8778 0)
 			(effects
 				(font
@@
 		)
 		(property "Value" "Side keys"
-			(at 39.878 76.1421 0)
+			(at 53.848 86.3021 0)
 			(effects
 				(font
@@
 		)
 		(property "Footprint" ""
-			(at 41.91 74.93 0)
+			(at 55.88 85.09 0)
 			(effects
 				(font
@@
 		)
 		(property "Datasheet" "~"
-			(at 41.91 74.93 0)
+			(at 55.88 85.09 0)
 			(effects
 				(font
@@
 		)
 		(property "Description" "Generic connector, single row, 01x05, script generated (kicad-library-utils/schlib/autogen/connector/)"
-			(at 41.91 74.93 0)
-			(effects
-				(font
+			(at 55.88 85.09 0)
+			(effects
+				(font
