File: keyboard.kicad_sch (KiCad schematic)
At the start: 6 parts, among them J6 Side keys, J7 Keyboard, Q3 BSS138

Commit message: Added keyboard connector to the layout
* Changed J7 connector from "01x16" to "01x16 with MP" variant
* Positioned J7 on the layout, bottom side
Parts:
- J7: footprint (none) -> parts:FPC-SMD_P0.50-16P_FGS-XJ-H2.0; symbol Connector_Generic:Conn_01x16 -> Connector_Generic_MountingPin:Conn_01x16_MountingPin; LCSC (none) -> C262665; MPN (none) -> AFC01-S16FCA-00
Connections:
- net GND: now also J7.MP (MountPin)
Changed lines of the file:
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@@
+	)
+	(junction
+		(at 130.81 119.38)
+		(diameter 0)
+		(color 0 0 0 0)
 	)
 	(junction
@@
 	(wire
 		(pts
+			(xy 130.81 119.38) (xy 130.81 120.65)
+		)
+		(stroke
+			(width 0)
+			(type default)
+		)
+	)
+	(wire
+		(pts
 			(xy 128.27 74.93) (xy 130.81 74.93)
 		)
@@
 	(wire
 		(pts
-			(xy 130.81 113.03) (xy 130.81 115.57)
+			(xy 130.81 113.03) (xy 130.81 119.38)
 		)
 		(stroke
@@
 	(wire
 		(pts
+			(xy 123.19 118.11) (xy 123.19 119.38)
+		)
+		(stroke
+			(width 0)
+			(type default)
+		)
+	)
+	(wire
+		(pts
 			(xy 128.27 85.09) (xy 135.89 85.09)
+		)
+		(stroke
+			(width 0)
+			(type default)
+		)
+	)
+	(wire
+		(pts
+			(xy 123.19 119.38) (xy 130.81 119.38)
 		)
 		(stroke
@@
 	(symbol
 		(lib_id "power:GND")
-		(at 130.81 115.57 0)
+		(at 130.81 120.65 0)
 		(unit 1)
 		(exclude_from_sim no)
@@
 		(fields_autoplaced yes)
 		(property "Reference" "#PWR071"
-			(at 130.81 121.92 0)
+			(at 130.81 127 0)
 			(effects
 				(font
@@
 		)
 		(property "Value" "GND"
-			(at 130.81 119.7031 0)
+			(at 130.81 124.7831 0)
 			(effects
 				(font
@@
 		)
 		(property "Footprint" ""
-			(at 130.81 115.57 0)
+			(at 130.81 120.65 0)
 			(effects
 				(font
@@
 		)
 		(property "Datasheet" ""
-			(at 130.81 115.57 0)
+			(at 130.81 120.65 0)
 			(effects
 				(font
@@
 		)
 		(property "Description" "Power symbol creates a global label with name \"GND\" , ground"
-			(at 130.81 115.57 0)
+			(at 130.81 120.65 0)
 			(effects
 				(font
@@
 	)
 	(symbol
-		(lib_id "Connector_Generic:Conn_01x16")
+		(lib_id "Connector_Generic_MountingPin:Conn_01x16_MountingPin")
 		(at 123.19 92.71 0)
 		(mirror y)
@@
 		(dnp no)
 		(property "Reference" "J7"
-			(at 123.19 118.4445 0)
+			(at 123.444 69.342 0)
 			(effects
 				(font
@@
 		)
 		(property "Value" "Keyboard"
-			(at 123.19 116.0202 0)
-			(effects
-				(font
-					(size 1.27 1.27)
-				)
-			)
-		)
-		(property "Footprint" ""
+			(at 123.19 71.7437 0)
+			(effects
+				(font
+					(size 1.27 1.27)
+				)
+			)
+		)
+		(property "Footprint" "parts:FPC-SMD_P0.50-16P_FGS-XJ-H2.0"
 			(at 123.19 92.71 0)
 			(effects
@@
 			)
 		)
-		(property "Description" "Generic connector, single row, 01x16, script generated (kicad-library-utils/schlib/autogen/connector/)"
+		(property "Description" "Generic connectable mounting pin connector, single row, 01x16, script generated (kicad-library-utils/schlib/autogen/connector/)"
 			(at 123.19 92.71 0)
 			(effects
@@
 			)
 		)
-		(property "MPN" ""
+		(property "MPN" "AFC01-S16FCA-00"
 			(at 123.19 92.71 0)
 			(effects
@@
 			)
 		)
+		(property "LCSC" "C262665"
+			(at 123.19 92.71 0)
+			(effects
+				(font
+					(size 1.27 1.27)
+				)
+				(hide yes)
+			)
+		)
 		(pin "1"
 		)
@@
 		(pin "5"
 		)
+		(pin "MP"
+		)
 		(instances

Commit message: Added footprint and positions for the side keys (BTN2/PTT)
* Pad footprint on the original PCB (Retevis C62) is 1.7x2.2 mm.
* Side keys are mounted on a separate PCB soldered via 5 pads on
  the main PCB.
Parts:
- removed J6: Side keys, symbol Connector_Generic:Conn_01x05
- added J11, J12, J15: GND, parts:Solder_Pad-1.7x2.2mm, symbol Connector_Generic:Conn_01x01
- added J13: PTT, parts:Solder_Pad-1.7x2.2mm, symbol Connector_Generic:Conn_01x01
- added J14: BTN_2, parts:Solder_Pad-1.7x2.2mm, symbol Connector_Generic:Conn_01x01
Connections:
- net GND: now also J11.1 (Pin_1), J12.1 (Pin_1), J15.1 (Pin_1)
- net SIDE_BTN: now also J14.1 (Pin_1)
- net SIDE_PTT: now also J13.1 (Pin_1)

Commit message: Fixed pinout for the SoM
* Added missing pin definitions in MCM-iMX93 symbol
* Added information about the keyboard wiring
* Assigned all signals to pins in the SoM
Changed lines of the file:
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@@
 		(members "D1" "D2" "D3" "D4" "D5" "D6" "D7" "D8" "D9")
+	)
+	(text_box "Original C62 keypad connected in matrix.\n* D1-D4 + D9 are rows\n* D5-D8 are columns"
+		(exclude_from_sim no)
+		(at 138.43 60.96 0)
+		(size 26.67 11.43)
+		(margins 0.9525 0.9525 0.9525 0.9525)
+		(stroke
+			(width 0)
+			(type solid)
+		)
+		(fill
+			(type none)
+		)
+		(effects
+			(font
+				(size 1.27 1.27)
+			)
+			(justify left)
+		)
 	)
 	(text_box "Solder pads for the side keys (buttons). These have their own PCB."

Commit message: updates
- updated the 5V line (diode connected sources - USB and DC/DC)
- proposed a power on-off circuit based on a XNOR gate
- reannotated the schematic
- updated the PDF
Parts:
- renumbered J15 to J10, J7 to J11, J11 to J6, J12 to J7, J13 to J8, J14 to J9, Q3 to Q4, R31 to R42, R32 to R43, R33 to R44
Changed lines of the file:
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@@
 	(title_block
 		(title "LinHT - Linux-based SDR handheld transceiver")
-		(date "13 July 2025")
+		(date "15 July 2025")
 		(rev "A")
 		(company "M17 Foundation")
@@
 		(dnp no)
 		(fields_autoplaced yes)
-		(property "Reference" "#PWR071"
+		(property "Reference" "#PWR092"
 			(at 130.81 127 0)
 			(effects
@@
 			(project ""
 				(path "/73efc1fc-21f6-4aef-9f73-508fe18fa32e/058c0cc5-75b0-4494-8e78-217aac2f1bdc"
-					(reference "#PWR071")
+					(reference "#PWR092")
 					(unit 1)
 				)
@@
 		(dnp no)
 		(fields_autoplaced yes)
-		(property "Reference" "R32"
+		(property "Reference" "R43"
 			(at 163.322 100.3878 0)
 			(effects
@@
 			(project "linht-hw"
 				(path "/73efc1fc-21f6-4aef-9f73-508fe18fa32e/058c0cc5-75b0-4494-8e78-217aac2f1bdc"
-					(reference "R32")
+					(reference "R43")
 					(unit 1)
 				)
@@
 		(dnp no)
 		(fields_autoplaced yes)
-		(property "Reference" "#PWR073"
+		(property "Reference" "#PWR094"
 			(at 165.1 113.03 0)
 			(effects
@@
 			(project "linht-hw"
 				(path "/73efc1fc-21f6-4aef-9f73-508fe18fa32e/058c0cc5-75b0-4494-8e78-217aac2f1bdc"
-					(reference "#PWR073")
+					(reference "#PWR094")
 					(unit 1)
 				)
@@
 		(on_board yes)
 		(dnp no)
-		(property "Reference" "J14"
+		(property "Reference" "J9"
 			(at 52.07 114.3 0)
 			(effects
@@
 			(project "linht-hw"
 				(path "/73efc1fc-21f6-4aef-9f73-508fe18fa32e/058c0cc5-75b0-4494-8e78-217aac2f1bdc"
-					(reference "J14")
+					(reference "J9")
 					(unit 1)
 				)
@@
 		(on_board yes)
 		(dnp no)
-		(property "Reference" "J15"
+		(property "Reference" "J10"
 			(at 52.07 118.11 0)
 			(effects
@@
 			(project "linht-hw"
 				(path "/73efc1fc-21f6-4aef-9f73-508fe18fa32e/058c0cc5-75b0-4494-8e78-217aac2f1bdc"
-					(reference "J15")
+					(reference "J10")
 					(unit 1)
 				)
@@
 		(dnp no)
 		(fields_autoplaced yes)
-		(property "Reference" "R31"
+		(property "Reference" "R42"
 			(at 156.718 82.6078 0)
 			(effects
@@
 			(project ""
 				(path "/73efc1fc-21f6-4aef-9f73-508fe18fa32e/058c0cc5-75b0-4494-8e78-217aac2f1bdc"
-					(reference "R31")
+					(reference "R42")
 					(unit 1)
 				)
@@
 		(dnp no)
 		(fields_autoplaced yes)
-		(property "Reference" "#PWR091"
+		(property "Reference" "#PWR089"
 			(at 71.12 104.14 0)
 			(effects
@@
 			(project "linht-hw"
 				(path "/73efc1fc-21f6-4aef-9f73-508fe18fa32e/058c0cc5-75b0-4494-8e78-217aac2f1bdc"
-					(reference "#PWR091")
+					(reference "#PWR089")
 					(unit 1)
 				)
@@
 		(dnp no)
 		(fields_autoplaced yes)
-		(property "Reference" "#PWR03"
+		(property "Reference" "#PWR090"
 			(at 71.12 118.11 0)
 			(effects
@@
 			(project "linht-hw"
 				(path "/73efc1fc-21f6-4aef-9f73-508fe18fa32e/058c0cc5-75b0-4494-8e78-217aac2f1bdc"
-					(reference "#PWR03")
+					(reference "#PWR090")
 					(unit 1)
 				)
@@
 		(dnp no)
 		(fields_autoplaced yes)
-		(property "Reference" "#PWR072"
+		(property "Reference" "#PWR093"
 			(at 154.94 113.03 0)
 			(effects
@@
 			(project "linht-hw"
 				(path "/73efc1fc-21f6-4aef-9f73-508fe18fa32e/058c0cc5-75b0-4494-8e78-217aac2f1bdc"
-					(reference "#PWR072")
+					(reference "#PWR093")
 					(unit 1)
 				)
@@
 		(dnp no)
 		(fields_autoplaced yes)
-		(property "Reference" "R33"
+		(property "Reference" "R44"
 			(at 171.45 90.0895 90)
 			(effects
@@
 			(project "linht-hw"
 				(path "/73efc1fc-21f6-4aef-9f73-508fe18fa32e/058c0cc5-75b0-4494-8e78-217aac2f1bdc"
-					(reference "R33")
+					(reference "R44")
 					(unit 1)
 				)
@@
 		(dnp no)
 		(fields_autoplaced yes)
-		(property "Reference" "#PWR070"
+		(property "Reference" "#PWR091"
 			(at 130.81 76.2 0)
 			(effects
@@
 			(project ""
 				(path "/73efc1fc-21f6-4aef-9f73-508fe18fa32e/058c0cc5-75b0-4494-8e78-217aac2f1bdc"
-					(reference "#PWR070")
+					(reference "#PWR091")
 					(unit 1)
 				)
@@
 		(on_board yes)
 		(dnp no)
-		(property "Reference" "J13"
+		(property "Reference" "J8"
 			(at 52.07 110.49 0)
 			(effects
@@
 			(project "linht-hw"
 				(path "/73efc1fc-21f6-4aef-9f73-508fe18fa32e/058c0cc5-75b0-4494-8e78-217aac2f1bdc"
-					(reference "J13")
+					(reference "J8")
 					(unit 1)
 				)
@@
 		(on_board yes)
 		(dnp no)
-		(property "Reference" "J11"
+		(property "Reference" "J6"
 			(at 52.07 100.33 0)
 			(effects
@@
 			(project ""
 				(path "/73efc1fc-21f6-4aef-9f73-508fe18fa32e/058c0cc5-75b0-4494-8e78-217aac2f1bdc"
-					(reference "J11")
+					(reference "J6")
 					(unit 1)
 				)
@@
 		(on_board yes)
 		(dnp no)
-		(property "Reference" "J7"
+		(property "Reference" "J11"
 			(at 123.444 69.342 0)
 			(effects
@@
 			(project ""
 				(path "/73efc1fc-21f6-4aef-9f73-508fe18fa32e/058c0cc5-75b0-4494-8e78-217aac2f1bdc"
-					(reference "J7")
+					(reference "J11")
 					(unit 1)
 				)
@@
 		(on_board yes)
 		(dnp no)
-		(property "Reference" "J12"
+		(property "Reference" "J7"
 			(at 52.07 104.14 0)
 			(effects
@@
 			(project "linht-hw"
 				(path "/73efc1fc-21f6-4aef-9f73-508fe18fa32e/058c0cc5-75b0-4494-8e78-217aac2f1bdc"
-					(reference "J12")
+					(reference "J7")
 					(unit 1)
 				)
@@
 		(on_board yes)
 		(dnp no)
-		(property "Reference" "Q3"
+		(property "Reference" "Q4"
 			(at 152.273 94.0378 0)
 			(effects
@@
 			(project ""
 				(path "/73efc1fc-21f6-4aef-9f73-508fe18fa32e/058c0cc5-75b0-4494-8e78-217aac2f1bdc"
-					(reference "Q3")
+					(reference "Q4")
 					(unit 1)
 				)

Commit message: tweaked the power-on circuit
- supplied the XNOR gate with 5V instead of 3.3V
- added a MOSFET to drive the 3.3V DC/DC converter's EN pin
- removed a pull-up resistor at the ON/OFF line
Parts:
- renumbered Q4 to Q5
Changed lines of the file:
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@@
 	(title_block
 		(title "LinHT - Linux-based SDR handheld transceiver")
-		(date "15 July 2025")
+		(date "17 July 2025")
 		(rev "A")
 		(company "M17 Foundation")
@@
 		(dnp no)
 		(fields_autoplaced yes)
-		(property "Reference" "#PWR092"
+		(property "Reference" "#PWR093"
 			(at 130.81 127 0)
 			(effects
@@
 			(project ""
 				(path "/73efc1fc-21f6-4aef-9f73-508fe18fa32e/058c0cc5-75b0-4494-8e78-217aac2f1bdc"
-					(reference "#PWR092")
+					(reference "#PWR093")
 					(unit 1)
 				)
@@
 		(dnp no)
 		(fields_autoplaced yes)
-		(property "Reference" "#PWR094"
+		(property "Reference" "#PWR095"
 			(at 165.1 113.03 0)
 			(effects
@@
 			(project "linht-hw"
 				(path "/73efc1fc-21f6-4aef-9f73-508fe18fa32e/058c0cc5-75b0-4494-8e78-217aac2f1bdc"
-					(reference "#PWR094")
+					(reference "#PWR095")
 					(unit 1)
 				)
@@
 		(dnp no)
 		(fields_autoplaced yes)
-		(property "Reference" "#PWR089"
+		(property "Reference" "#PWR090"
 			(at 71.12 104.14 0)
 			(effects
@@
 			(project "linht-hw"
 				(path "/73efc1fc-21f6-4aef-9f73-508fe18fa32e/058c0cc5-75b0-4494-8e78-217aac2f1bdc"
-					(reference "#PWR089")
+					(reference "#PWR090")
 					(unit 1)
 				)
@@
 		(dnp no)
 		(fields_autoplaced yes)
-		(property "Reference" "#PWR090"
+		(property "Reference" "#PWR091"
 			(at 71.12 118.11 0)
 			(effects
@@
 			(project "linht-hw"
 				(path "/73efc1fc-21f6-4aef-9f73-508fe18fa32e/058c0cc5-75b0-4494-8e78-217aac2f1bdc"
-					(reference "#PWR090")
+					(reference "#PWR091")
 					(unit 1)
 				)
@@
 		(dnp no)
 		(fields_autoplaced yes)
-		(property "Reference" "#PWR093"
+		(property "Reference" "#PWR094"
 			(at 154.94 113.03 0)
 			(effects
@@
 			(project "linht-hw"
 				(path "/73efc1fc-21f6-4aef-9f73-508fe18fa32e/058c0cc5-75b0-4494-8e78-217aac2f1bdc"
-					(reference "#PWR093")
+					(reference "#PWR094")
 					(unit 1)
 				)
@@
 		(dnp no)
 		(fields_autoplaced yes)
-		(property "Reference" "#PWR091"
+		(property "Reference" "#PWR092"
 			(at 130.81 76.2 0)
 			(effects
@@
 			(project ""
 				(path "/73efc1fc-21f6-4aef-9f73-508fe18fa32e/058c0cc5-75b0-4494-8e78-217aac2f1bdc"
-					(reference "#PWR091")
+					(reference "#PWR092")
 					(unit 1)
 				)
@@
 		(on_board yes)
 		(dnp no)
-		(property "Reference" "Q4"
+		(property "Reference" "Q5"
 			(at 152.273 94.0378 0)
 			(effects
@@
 			(project ""
 				(path "/73efc1fc-21f6-4aef-9f73-508fe18fa32e/058c0cc5-75b0-4494-8e78-217aac2f1bdc"
-					(reference "Q4")
+					(reference "Q5")
 					(unit 1)
 				)

Commit message: minor power on/off circuit tweaks
Parts:
- renumbered R42 to R43, R43 to R44, R44 to R45
Changed lines of the file:
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@@
 		(dnp no)
 		(fields_autoplaced yes)
-		(property "Reference" "R43"
+		(property "Reference" "R44"
 			(at 163.322 100.3878 0)
 			(effects
@@
 			(project "linht-hw"
 				(path "/73efc1fc-21f6-4aef-9f73-508fe18fa32e/058c0cc5-75b0-4494-8e78-217aac2f1bdc"
-					(reference "R43")
+					(reference "R44")
 					(unit 1)
 				)
@@
 		(dnp no)
 		(fields_autoplaced yes)
-		(property "Reference" "R42"
+		(property "Reference" "R43"
 			(at 156.718 82.6078 0)
 			(effects
@@
 			(project ""
 				(path "/73efc1fc-21f6-4aef-9f73-508fe18fa32e/058c0cc5-75b0-4494-8e78-217aac2f1bdc"
-					(reference "R42")
+					(reference "R43")
 					(unit 1)
 				)
@@
 		(dnp no)
 		(fields_autoplaced yes)
-		(property "Reference" "R44"
+		(property "Reference" "R45"
 			(at 171.45 90.0895 90)
 			(effects
@@
 			(project "linht-hw"
 				(path "/73efc1fc-21f6-4aef-9f73-508fe18fa32e/058c0cc5-75b0-4494-8e78-217aac2f1bdc"
-					(reference "R44")
-					(unit 1)
-				)
+					(reference "R45")
+					(unit 1)
+				)
