File: keyboard.kicad_sch (KiCad schematic)
At the start: 10 parts, among them J10 GND, J11 Keyboard, J6 GND, J7 GND, J8 PTT, J9 BTN_2, Q5 BSS138

Commit message: Added BOM assigment for most of the parts
Parts:
- Q5: LCSC (none) -> C40912; MPN (none) -> BSS138-7-F; PN (none) -> 621-BSS138-7-F
- R43: LCSC (none) -> C542965; PN (none) -> ERJPA2F1500X
- R44: LCSC (none) -> C25792; PN (none) -> 0402WGF4702TCE
- R45: LCSC (none) -> C25076; PN (none) -> 0402WGF1000TCE
Changed lines of the file:
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@@
+			)
+		)
+		(property "LCSC" "C25792"
+			(at 165.1 101.6 0)
+			(effects
+				(font
+					(size 1.27 1.27)
+				)
+				(hide yes)
+			)
+		)
+		(property "PN" "0402WGF4702TCE"
+			(at 165.1 101.6 0)
+			(effects
+				(font
+					(size 1.27 1.27)
+				)
+				(hide yes)
 			)
 		)
@@
 			)
 		)
+		(property "LCSC" "C542965"
+			(at 154.94 83.82 0)
+			(effects
+				(font
+					(size 1.27 1.27)
+				)
+				(hide yes)
+			)
+		)
+		(property "PN" "ERJPA2F1500X"
+			(at 154.94 83.82 0)
+			(effects
+				(font
+					(size 1.27 1.27)
+				)
+				(hide yes)
+			)
+		)
 		(pin "1"
 		)
@@
 			)
 		)
+		(property "LCSC" "C25076"
+			(at 171.45 95.25 90)
+			(effects
+				(font
+					(size 1.27 1.27)
+				)
+				(hide yes)
+			)
+		)
+		(property "PN" "0402WGF1000TCE"
+			(at 171.45 95.25 90)
+			(effects
+				(font
+					(size 1.27 1.27)
+				)
+				(hide yes)
+			)
+		)
 		(pin "1"
 		)
@@
 			(at 157.48 95.25 0)
 			(effects
+				(font
+					(size 1.27 1.27)
+				)
+				(hide yes)
+			)
+		)
+		(property "LCSC" "C40912"
+			(at 157.48 95.25 0)
+			(effects
+				(font
+					(size 1.27 1.27)
+				)
+				(hide yes)
+			)
+		)
+		(property "MPN" "BSS138-7-F"
+			(at 157.48 95.25 0)
+			(effects
+				(font
+					(size 1.27 1.27)
+				)
+				(hide yes)
+			)
+		)
+		(property "PN" " 621-BSS138-7-F "
+			(at 157.48 95.25 0)
+			(effects
