File: linht-hw.kicad_sch (KiCad schematic)
At the start: 0 parts

Commit message: Replaced WM8960 to the newer TLV320AIC3100
WM8960 is obsolete, so this change is needed.
Fixes #29
Other:
- sheet Audio ports: added MIC_EXT; removed JACK_DETECT, MIC_GAIN, ~{MIC_MUTE}
- sheet Connectors ports: added JACK_DETECT; removed MIC_IN, SPK_OUT
- sheet SoC ports: added JACK_DETECT; removed MIC_GAIN, ~{MIC_MUTE}
Changed lines of the file:
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@@
-	(wire
-		(pts
-			(xy 113.03 134.62) (xy 176.53 134.62)
-		)
-		(stroke
-			(width 0)
-			(type default)
-		)
-	)
 	(wire
 		(pts
@@
 	(wire
 		(pts
+			(xy 77.47 137.16) (xy 87.63 137.16)
+		)
+		(stroke
+			(width 0)
+			(type default)
+		)
+	)
+	(wire
+		(pts
 			(xy 163.83 93.98) (xy 176.53 93.98)
 		)
@@
 	(wire
 		(pts
-			(xy 77.47 156.21) (xy 176.53 156.21)
-		)
-		(stroke
-			(width 0)
-			(type default)
-		)
-	)
-	(wire
-		(pts
 			(xy 121.92 76.2) (xy 121.92 86.36)
 		)
@@
 	(wire
 		(pts
-			(xy 113.03 99.06) (xy 127 99.06)
-		)
-		(stroke
-			(width 0)
-			(type default)
-		)
-	)
-	(wire
-		(pts
 			(xy 163.83 114.3) (xy 176.53 114.3)
 		)
@@
 	(wire
 		(pts
+			(xy 163.83 124.46) (xy 176.53 124.46)
+		)
+		(stroke
+			(width 0)
+			(type default)
+		)
+	)
+	(wire
+		(pts
 			(xy 163.83 46.99) (xy 176.53 46.99)
 		)
@@
 	(wire
 		(pts
-			(xy 77.47 80.01) (xy 77.47 156.21)
+			(xy 77.47 80.01) (xy 77.47 137.16)
 		)
 		(stroke
@@
 		(pts
 			(xy 163.83 44.45) (xy 176.53 44.45)
-		)
-		(stroke
-			(width 0)
-			(type default)
-		)
-	)
-	(wire
-		(pts
-			(xy 113.03 101.6) (xy 127 101.6)
 		)
 		(stroke
@@
 	(sheet
 		(at 176.53 88.9)
-		(size 25.4 71.12)
+		(size 25.4 53.975)
 		(exclude_from_sim no)
 		(in_bom yes)
@@
 		)
 		(property "Sheetfile" "connectors.kicad_sch"
-			(at 176.53 160.6046 0)
+			(at 176.53 143.4596 0)
 			(effects
 				(font
@@
 			)
 		)
-		(pin "MIC_IN" input
-			(at 176.53 156.21 180)
-			(effects
-				(font
-					(size 1.27 1.27)
-				)
-				(justify left)
-			)
-		)
 		(pin "MIC_OUT" output
 			(at 176.53 139.7 180)
@@
 			)
 		)
-		(pin "SPK_OUT" output
-			(at 176.53 134.62 180)
-			(effects
-				(font
-					(size 1.27 1.27)
-				)
-				(justify left)
-			)
-		)
 		(pin "USB_DN" bidirectional
 			(at 176.53 109.22 180)
@@
 				)
 				(justify right)
+			)
+		)
+		(pin "JACK_DETECT" output
+			(at 176.53 124.46 180)
+			(effects
+				(font
+					(size 1.27 1.27)
+				)
+				(justify left)
 			)
 		)
@@
 			)
 		)
-		(pin "MIC_GAIN" output
-			(at 127 99.06 180)
-			(effects
-				(font
-					(size 1.27 1.27)
-				)
-				(justify left)
-			)
-		)
-		(pin "~{MIC_MUTE}" output
-			(at 127 101.6 180)
-			(effects
-				(font
-					(size 1.27 1.27)
-				)
-				(justify left)
-			)
-		)
 		(pin "EXT_PTT" input
 			(at 163.83 97.79 0)
@@
 		(pin "VOL_BATT" input
 			(at 163.83 80.01 0)
+			(effects
+				(font
+					(size 1.27 1.27)
+				)
+				(justify right)
+			)
+		)
+		(pin "JACK_DETECT" input
+			(at 163.83 124.46 0)
 			(effects
 				(font
@@
 			)
 		)
-		(pin "MIC_GAIN" input
-			(at 113.03 99.06 0)
-			(effects
-				(font
-					(size 1.27 1.27)
-				)
-				(justify right)
-			)
-		)
 		(pin "MIC_IN" input
-			(at 113.03 139.7 0)
-			(effects
-				(font
-					(size 1.27 1.27)
-				)
-				(justify right)
-			)
-		)
-		(pin "~{MIC_MUTE}" input
-			(at 113.03 101.6 0)
-			(effects
-				(font
-					(size 1.27 1.27)
-				)
-				(justify right)
+			(at 87.63 137.16 180)
+			(effects
+				(font
+					(size 1.27 1.27)
+				)
+				(justify left)
 			)
 		)
@@
 			)
 		)
-		(pin "JACK_DETECT" input
-			(at 113.03 134.62 0)
-			(effects
-				(font
-					(size 1.27 1.27)
-				)
-				(justify right)
-			)
-		)
 		(pin "SPK_OUT" output
 			(at 113.03 137.16 0)
 			(effects
 				(font
+					(size 1.27 1.27)
+				)
+				(justify right)
+			)
+		)
+		(pin "MIC_EXT" input
+			(at 113.03 139.7 0)
+			(effects
+				(font

Commit message: Improved schematics readability
Other:
- sheet Audio ports: added MIC_INT; removed MIC_IN
Changed lines of the file:
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@@
 	(wire
 		(pts
-			(xy 77.47 137.16) (xy 87.63 137.16)
+			(xy 77.47 139.7) (xy 87.63 139.7)
 		)
 		(stroke
@@
 	(wire
 		(pts
-			(xy 77.47 80.01) (xy 77.47 137.16)
+			(xy 77.47 80.01) (xy 77.47 139.7)
 		)
 		(stroke
@@
 		)
 		(fill
-			(color 0 0 0 0.0000)
+			(color 255 255 194 1.0000)
 		)
 		(property "Sheetname" "Keyboard"
@@
 		)
 		(fill
-			(color 0 0 0 0.0000)
+			(color 255 255 194 1.0000)
 		)
 		(property "Sheetname" "RF"
@@
 		)
 		(fill
-			(color 0 0 0 0.0000)
+			(color 255 255 194 1.0000)
 		)
 		(property "Sheetname" "Display"
@@
 		)
 		(fill
-			(color 0 0 0 0.0000)
+			(color 255 255 194 1.0000)
 		)
 		(property "Sheetname" "Connectors"
@@
 		)
 		(fill
-			(color 0 0 0 0.0000)
+			(color 255 255 194 1.0000)
 		)
 		(property "Sheetname" "SoC"
@@
 		)
 		(fill
-			(color 0 0 0 0.0000)
+			(color 255 255 194 1.0000)
 		)
 		(property "Sheetname" "Power"
@@
 		)
 		(fill
-			(color 0 0 0 0.0000)
+			(color 255 255 194 1.0000)
 		)
 		(property "Sheetname" "Audio"
@@
 			)
 		)
-		(pin "MIC_IN" input
-			(at 87.63 137.16 180)
-			(effects
-				(font
+		(pin "MIC_INT" input
+			(at 87.63 139.7 180)
+			(effects
+				(font

Commit message: [WIP] Added an RF PA based on GRF5604
Fixes #27
Other:
- sheet RF ports: added RF_PA_SHUTDOWN; removed none
Changed lines of the file:
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@@
+			)
+		)
+		(pin "RF_PA_SHUTDOWN" input
+			(at 176.53 54.61 180)
+			(effects
+				(font
+					(size 1.27 1.27)
+				)
+				(justify left)
 			)
 		)
