File: linht-hw.kicad_sch (KiCad schematic)
At the start: 2 parts

Commit message: Removed battery voltage divider and `U_BATT_MON` signal to SoM
Battery voltage can and will be measured by the BQ25792RQ IC via I2C
register.
Other:
- sheet Power ports: added none; removed U_BATT_MON
Changed lines of the file:
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@@
-	(wire
-		(pts
-			(xy 163.83 80.01) (xy 212.09 80.01)
-		)
-		(stroke
-			(width 0)
-			(type default)
-		)
-	)
 	(wire
 		(pts
@@
 			)
 		)
-		(pin "U_BATT_MON" output
-			(at 212.09 80.01 180)
-			(effects
-				(font
-					(size 1.27 1.27)
-				)
-				(justify left)
-			)
-		)

Commit message: Added power management ATTiny826
Fixes #32
Fixes #35
Fixes #23
Connections:
- no-connect marks 2 -> 1
Other:
- sheet Power ports: added SIDE_BTN, USB_BOOT; removed 3V3_ON_REQ
- sheet SoC ports: added none; removed 3V3_ON_REQ, ON/OFF_SW, VOL_BATT
Changed lines of the file:
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@@
-	)
-	(junction
-		(at 121.92 86.36)
-		(diameter 0)
-		(color 0 0 0 0)
 	)
 	(junction
@@
 		(at 127 52.07)
 	)
-	(no_connect
-		(at 127 73.66)
-	)
 	(wire
 		(pts
@@
 	(wire
 		(pts
-			(xy 207.01 102.87) (xy 201.93 102.87)
+			(xy 207.01 100.33) (xy 201.93 100.33)
 		)
 		(stroke
@@
 	(wire
 		(pts
+			(xy 163.83 80.01) (xy 212.09 80.01)
+		)
+		(stroke
+			(width 0)
+			(type default)
+		)
+	)
+	(wire
+		(pts
 			(xy 113.03 55.88) (xy 127 55.88)
 		)
@@
 	(wire
 		(pts
-			(xy 121.92 76.2) (xy 121.92 86.36)
-		)
-		(stroke
-			(width 0)
-			(type default)
-		)
-	)
-	(wire
-		(pts
-			(xy 113.03 86.36) (xy 121.92 86.36)
+			(xy 113.03 86.36) (xy 127 86.36)
 		)
 		(stroke
@@
 	(wire
 		(pts
+			(xy 200.66 77.47) (xy 212.09 77.47)
+		)
+		(stroke
+			(width 0)
+			(type default)
+		)
+	)
+	(wire
+		(pts
 			(xy 163.83 46.99) (xy 176.53 46.99)
 		)
@@
 	(wire
 		(pts
-			(xy 207.01 90.17) (xy 207.01 102.87)
+			(xy 207.01 87.63) (xy 207.01 100.33)
 		)
 		(stroke
@@
 	(wire
 		(pts
-			(xy 127 76.2) (xy 121.92 76.2)
-		)
-		(stroke
-			(width 0)
-			(type default)
-		)
-	)
-	(wire
-		(pts
 			(xy 113.03 111.76) (xy 127 111.76)
 		)
@@
 	(wire
 		(pts
-			(xy 121.92 86.36) (xy 127 86.36)
-		)
-		(stroke
-			(width 0)
-			(type default)
-		)
-	)
-	(wire
-		(pts
 			(xy 113.03 139.7) (xy 176.53 139.7)
 		)
@@
 		)
 	)
+	(wire
+		(pts
+			(xy 163.83 85.09) (xy 212.09 85.09)
+		)
+		(stroke
+			(width 0)
+			(type default)
+		)
+	)
 	(bus
 		(pts
@@
 	(wire
 		(pts
-			(xy 212.09 90.17) (xy 207.01 90.17)
+			(xy 212.09 87.63) (xy 207.01 87.63)
 		)
 		(stroke
@@
 	(wire
 		(pts
-			(xy 163.83 85.09) (xy 212.09 85.09)
-		)
-		(stroke
-			(width 0)
-			(type default)
-		)
-	)
-	(wire
-		(pts
 			(xy 248.92 72.39) (xy 248.92 69.85)
 		)
@@
 			(width 0)
 			(type default)
+		)
+	)
+	(label "SIDE_BTN"
+		(at 200.66 77.47 0)
+		(effects
+			(font
+				(size 1.27 1.27)
+			)
+			(justify left bottom)
 		)
 	)
@@
 	(label "I2C_SCL"
 		(at 116.84 105.41 0)
+		(effects
+			(font
+				(size 1.27 1.27)
+			)
+			(justify left bottom)
+		)
+	)
+	(label "SIDE_BTN"
+		(at 115.57 86.36 0)
 		(effects
 			(font
@@
 		)
 		(pin "SWITCH_ON_OFF" output
-			(at 201.93 102.87 0)
+			(at 201.93 100.33 0)
 			(effects
 				(font
@@
 		)
 		(pin "STBY" output
-			(at 163.83 87.63 0)
+			(at 163.83 85.09 0)
 			(effects
 				(font
@@
 		)
 		(pin "USB_BOOT" input
-			(at 127 76.2 180)
-			(effects
-				(font
-					(size 1.27 1.27)
-				)
-				(justify left)
+			(at 163.83 80.01 0)
+			(effects
+				(font
+					(size 1.27 1.27)
+				)
+				(justify right)
 			)
 		)
@@
 		)
 		(pin "~{RST}" input
-			(at 127 73.66 180)
-			(effects
-				(font
-					(size 1.27 1.27)
-				)
-				(justify left)
+			(at 163.83 77.47 0)
+			(effects
+				(font
+					(size 1.27 1.27)
+				)
+				(justify right)
 			)
 		)
@@
 			)
 		)
-		(pin "ON{slash}OFF_SW" input
-			(at 163.83 77.47 0)
-			(effects
-				(font
-					(size 1.27 1.27)
-				)
-				(justify right)
-			)
-		)
 		(pin "VOL_POT" input
 			(at 163.83 121.92 0)
@@
 			)
 		)
-		(pin "VOL_BATT" input
-			(at 163.83 80.01 0)
-			(effects
-				(font
-					(size 1.27 1.27)
-				)
-				(justify right)
-			)
-		)
 		(pin "JACK_DETECT" input
 			(at 163.83 124.46 0)
-			(effects
-				(font
-					(size 1.27 1.27)
-				)
-				(justify right)
-			)
-		)
-		(pin "3V3_ON_REQ" output
-			(at 163.83 85.09 0)
 			(effects
 				(font
@@
 	)
 	(sheet
-		(at 212.09 76.2)
-		(size 25.4 24.765)
+		(at 212.09 74.93)
+		(size 25.4 26.035)
 		(exclude_from_sim no)
 		(in_bom yes)
@@
 		)
 		(property "Sheetname" "Power"
-			(at 212.09 75.4884 0)
+			(at 212.09 74.2184 0)
 			(effects
 				(font
@@
 			)
 		)
-		(pin "3V3_ON_REQ" input
+		(pin "~{5V_ON_REQ}" input
+			(at 212.09 87.63 180)
+			(effects
+				(font
+					(size 1.27 1.27)
+				)
+				(justify left)
+			)
+		)
+		(pin "~{5V_OFF_REQ}" input
 			(at 212.09 85.09 180)
-			(effects
-				(font
-					(size 1.27 1.27)
-				)
-				(justify left)
-			)
-		)
-		(pin "~{5V_ON_REQ}" input
-			(at 212.09 90.17 180)
-			(effects
-				(font
-					(size 1.27 1.27)
-				)
-				(justify left)
-			)
-		)
-		(pin "~{5V_OFF_REQ}" input
-			(at 212.09 87.63 180)
 			(effects
 				(font
@@
 			(effects
 				(font
+					(size 1.27 1.27)
+				)
+				(justify left)
+			)
+		)
+		(pin "USB_BOOT" output
+			(at 212.09 80.01 180)
+			(effects
+				(font
+					(size 1.27 1.27)
+				)
+				(justify left)
+			)
+		)
+		(pin "SIDE_BTN" input
+			(at 212.09 77.47 180)
+			(effects
+				(font

Commit message: Minor schematics tweaks and pinout optimizations
Other:
- sheet Power ports: added SOM_RST; removed none
Changed lines of the file:
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@@
 	(wire
 		(pts
-			(xy 200.66 77.47) (xy 212.09 77.47)
+			(xy 203.2 74.93) (xy 212.09 74.93)
 		)
 		(stroke
@@
 	(wire
 		(pts
+			(xy 163.83 77.47) (xy 212.09 77.47)
+		)
+		(stroke
+			(width 0)
+			(type default)
+		)
+	)
+	(wire
+		(pts
 			(xy 248.92 72.39) (xy 248.92 69.85)
 		)
@@
 	)
 	(label "SIDE_BTN"
-		(at 200.66 77.47 0)
+		(at 203.2 74.93 0)
 		(effects
 			(font
@@
 	)
 	(sheet
-		(at 212.09 74.93)
-		(size 25.4 26.035)
+		(at 212.09 72.39)
+		(size 25.4 28.575)
 		(exclude_from_sim no)
 		(in_bom yes)
@@
 		)
 		(property "Sheetname" "Power"
-			(at 212.09 74.2184 0)
+			(at 212.09 71.6784 0)
 			(effects
 				(font
@@
 		)
 		(pin "SIDE_BTN" input
+			(at 212.09 74.93 180)
+			(effects
+				(font
+					(size 1.27 1.27)
+				)
+				(justify left)
+			)
+		)
+		(pin "SOM_RST" output
 			(at 212.09 77.47 180)
 			(effects

Commit message: Connected attenuator data signals to SoM and minor changes to SoM pinout
KBD_PWM from 105  -> 95  (GPIO2_IO[25])
RF_SW_CTRL from 104 -> 103 (GPIO2_IO[15])
RF_ATT_DATA to 107 (SPI7_SOUT)
RF_ATT_CLK to 106 (SPI7_SCK)
RF_ATT_LE1 to 105 (GPIO2_IO[12])
RF_ATT_LE2 to 104 (GPIO2_IO[13])
RF_PA_SHUTDOWN not decided yet
Other:
- sheet SoC ports: added RF_ATT_CLK, RF_ATT_DATA, RF_ATT_LE1, RF_ATT_LE2; removed none
- moved on the sheet: R25, R26
