File: audio.kicad_sch (KiCad schematic)
At the start: 44 parts, among them J3 Speaker, J4 GND spring, U3 MAX9814, U6 WM8960

Commit message: updates
- updated the 5V line (diode connected sources - USB and DC/DC)
- proposed a power on-off circuit based on a XNOR gate
- reannotated the schematic
- updated the PDF
Parts:
- renumbered C32 to C33, C33 to C34, C24 to C35, C25 to C36, C27 to C37, C30 to C38, C17 to C39, C18 to C40, C22 to C41, C23 to C42, C20 to C43, C49 to C44, C21 to C45, C48 to C46, C19 to C47, C47 to C48, C46 to C49, C55 to C50, C56 to C51, C44 to C52, C50 to C53, C28 to C54, C29 to C55, C45 to C56, C31 to C57, FB3 to FB2, J4 to J3, J3 to J4, R16 to R24, R19 to R25, R40 to R26, R15 to R27, R17 to R28, R18 to R29, R20 to R30, R41 to R31, TP8 to TP1, TP5 to TP2, TP6 to TP3, TP2 to TP4, TP3 to TP5, U3 to U7

Commit message: tweaked the power-on circuit
- supplied the XNOR gate with 5V instead of 3.3V
- added a MOSFET to drive the 3.3V DC/DC converter's EN pin
- removed a pull-up resistor at the ON/OFF line
Parts:
- renumbered C33 to C34, C34 to C35, C35 to C36, C36 to C37, C37 to C38, C38 to C39, C39 to C40, C40 to C41, C41 to C42, C42 to C43, C43 to C44, C44 to C45, C45 to C46, C46 to C47, C47 to C48, C48 to C49, C49 to C50, C50 to C51, C51 to C52, C52 to C53, C53 to C54, C54 to C55, C55 to C56, C56 to C57, C57 to C58

Commit message: minor power on/off circuit tweaks
Parts:
- renumbered R24 to R25, R25 to R26, R26 to R27, R27 to R28, R28 to R29, R29 to R30, R30 to R31, R31 to R32
Changed lines of the file:
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@@
 		(on_board yes)
 		(dnp no)
-		(property "Reference" "R24"
+		(property "Reference" "R25"
 			(at 69.342 94.234 0)
 			(effects
@@
 			(project "linht-hw"
 				(path "/73efc1fc-21f6-4aef-9f73-508fe18fa32e/c40b23ce-765e-4258-88c6-173a78d6d517"
-					(reference "R24")
+					(reference "R25")
 					(unit 1)
 				)
@@
 		(dnp no)
 		(fields_autoplaced yes)
-		(property "Reference" "R31"
+		(property "Reference" "R32"
 			(at 213.5887 80.3715 0)
 			(effects
@@
 			(project "linht-hw"
 				(path "/73efc1fc-21f6-4aef-9f73-508fe18fa32e/c40b23ce-765e-4258-88c6-173a78d6d517"
-					(reference "R31")
+					(reference "R32")
 					(unit 1)
 				)
@@
 		(on_board yes)
 		(dnp no)
-		(property "Reference" "R25"
+		(property "Reference" "R26"
 			(at 75.692 94.234 0)
 			(effects
@@
 			(project "linht-hw"
 				(path "/73efc1fc-21f6-4aef-9f73-508fe18fa32e/c40b23ce-765e-4258-88c6-173a78d6d517"
-					(reference "R25")
+					(reference "R26")
 					(unit 1)
 				)
@@
 		(on_board yes)
 		(dnp yes)
-		(property "Reference" "R26"
+		(property "Reference" "R27"
 			(at 98.552 86.36 90)
 			(effects
@@
 			(project "linht-hw"
 				(path "/73efc1fc-21f6-4aef-9f73-508fe18fa32e/c40b23ce-765e-4258-88c6-173a78d6d517"
-					(reference "R26")
+					(reference "R27")
 					(unit 1)
 				)
@@
 		(on_board yes)
 		(dnp no)
-		(property "Reference" "R29"
+		(property "Reference" "R30"
 			(at 124.46 138.8068 90)
 			(effects
@@
 			(project "linht-hw"
 				(path "/73efc1fc-21f6-4aef-9f73-508fe18fa32e/c40b23ce-765e-4258-88c6-173a78d6d517"
-					(reference "R29")
+					(reference "R30")
 					(unit 1)
 				)
@@
 		(dnp no)
 		(fields_autoplaced yes)
-		(property "Reference" "R28"
+		(property "Reference" "R29"
 			(at 120.8787 156.5715 0)
 			(effects
@@
 			(project "linht-hw"
 				(path "/73efc1fc-21f6-4aef-9f73-508fe18fa32e/c40b23ce-765e-4258-88c6-173a78d6d517"
-					(reference "R28")
+					(reference "R29")
 					(unit 1)
 				)
@@
 		(dnp no)
 		(fields_autoplaced yes)
-		(property "Reference" "R27"
+		(property "Reference" "R28"
 			(at 96.7487 138.7915 0)
 			(effects
@@
 			(project "linht-hw"
 				(path "/73efc1fc-21f6-4aef-9f73-508fe18fa32e/c40b23ce-765e-4258-88c6-173a78d6d517"
-					(reference "R27")
+					(reference "R28")
 					(unit 1)
 				)
@@
 		(on_board yes)
 		(dnp no)
-		(property "Reference" "R30"
+		(property "Reference" "R31"
 			(at 191.77 142.24 90)
 			(effects
@@
 			(project "linht-hw"
 				(path "/73efc1fc-21f6-4aef-9f73-508fe18fa32e/c40b23ce-765e-4258-88c6-173a78d6d517"
-					(reference "R30")
+					(reference "R31")
 					(unit 1)
 				)

Commit message: update
- brought some order to page 1
- routed on/off signals
-added SoM pin #10
- rendered PDF
Parts:
- added C60: 100n, Capacitor_SMD:C_0402_1005Metric, symbol Device:C_Small
- added R49: ?R, Resistor_SMD:R_0402_1005Metric, symbol Device:R_Small
- added RV1: ?R, symbol Device:R_Potentiometer
Connections:
- net GND: now also C60.2, RV1.1
- net VDD: now also C60.1, R49.1
- new net: R49.2, RV1.3
- new net VOL_POT: RV1.2
Other:
- moved on the sheet: J3
