File: connectors.kicad_sch (KiCad schematic)
At the start: 19 parts, among them J10 3.5mm, J8 USB_C, J9 2.5mm, U4 USBLC6-2SC6

Commit message: updates
- updated the 5V line (diode connected sources - USB and DC/DC)
- proposed a power on-off circuit based on a XNOR gate
- reannotated the schematic
- updated the PDF
Parts:
- renumbered D4 to D5, FB2 to FB3, H6 to H10, H10 to H2, H2 to H3, H9 to H4, H3 to H5, H8 to H6, H4 to H7, H7 to H8, H5 to H9, J8 to J12, J9 to J13, J10 to J14, R34 to R45, R35 to R46, R36 to R47, U4 to U8
Connections:
- net VBUS renamed +5V

Commit message: Assigned footprint and layout position of the 2.5 mm jack
Parts:
- J13: footprint (none) -> parts:Jack_2.5mm_PJ-204_Horizontal
Changed lines of the file:
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@@
 			)
 		)
-		(property "Footprint" ""
+		(property "Footprint" "parts:Jack_2.5mm_PJ-204_Horizontal"
 			(at 196.85 74.93 0)
 			(effects

Commit message: tweaked the power-on circuit
- supplied the XNOR gate with 5V instead of 3.3V
- added a MOSFET to drive the 3.3V DC/DC converter's EN pin
- removed a pull-up resistor at the ON/OFF line
Parts:
- renumbered D5 to D6
Changed lines of the file:
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@@
 	(title_block
 		(title "LinHT - Linux-based SDR handheld transceiver")
-		(date "15 July 2025")
+		(date "17 July 2025")
 		(rev "A")
 		(company "M17 Foundation")
@@
 		(dnp no)
 		(fields_autoplaced yes)
-		(property "Reference" "#PWR099"
+		(property "Reference" "#PWR0100"
 			(at 91.44 80.01 0)
 			(effects
@@
 			(project "linht-hw"
 				(path "/73efc1fc-21f6-4aef-9f73-508fe18fa32e/5f168690-b6ac-4b3d-aad0-4e97277dc85d"
-					(reference "#PWR099")
+					(reference "#PWR0100")
 					(unit 1)
 				)
@@
 		(on_board yes)
 		(dnp no)
-		(property "Reference" "#PWR097"
+		(property "Reference" "#PWR098"
 			(at 66.04 153.67 0)
 			(effects
@@
 			(project "linht-hw"
 				(path "/73efc1fc-21f6-4aef-9f73-508fe18fa32e/5f168690-b6ac-4b3d-aad0-4e97277dc85d"
-					(reference "#PWR097")
+					(reference "#PWR098")
 					(unit 1)
 				)
@@
 		(dnp no)
 		(fields_autoplaced yes)
-		(property "Reference" "D5"
+		(property "Reference" "D6"
 			(at 61.2775 129.54 0)
 			(effects
@@
 			(project "linht-hw"
 				(path "/73efc1fc-21f6-4aef-9f73-508fe18fa32e/5f168690-b6ac-4b3d-aad0-4e97277dc85d"
-					(reference "D5")
+					(reference "D6")
 					(unit 1)
 				)
@@
 		(on_board yes)
 		(dnp no)
-		(property "Reference" "#PWR096"
+		(property "Reference" "#PWR097"
 			(at 71.12 142.24 0)
 			(effects
@@
 			(project "linht-hw"
 				(path "/73efc1fc-21f6-4aef-9f73-508fe18fa32e/5f168690-b6ac-4b3d-aad0-4e97277dc85d"
-					(reference "#PWR096")
+					(reference "#PWR097")
 					(unit 1)
 				)
@@
 		(dnp no)
 		(fields_autoplaced yes)
-		(property "Reference" "#PWR098"
+		(property "Reference" "#PWR099"
 			(at 77.47 137.16 0)
 			(effects
@@
 			(project "linht-hw"
 				(path "/73efc1fc-21f6-4aef-9f73-508fe18fa32e/5f168690-b6ac-4b3d-aad0-4e97277dc85d"
-					(reference "#PWR098")
+					(reference "#PWR099")
 					(unit 1)
 				)
@@
 		(on_board yes)
 		(dnp no)
-		(property "Reference" "#PWR095"
+		(property "Reference" "#PWR096"
 			(at 39.37 182.88 0)
 			(effects
@@
 			(project "linht-hw"
 				(path "/73efc1fc-21f6-4aef-9f73-508fe18fa32e/5f168690-b6ac-4b3d-aad0-4e97277dc85d"
-					(reference "#PWR095")
+					(reference "#PWR096")
 					(unit 1)
 				)
@@
 		(dnp no)
 		(fields_autoplaced yes)
-		(property "Reference" "#PWR0101"
+		(property "Reference" "#PWR0102"
 			(at 189.23 86.36 0)
 			(effects
@@
 			(project ""
 				(path "/73efc1fc-21f6-4aef-9f73-508fe18fa32e/5f168690-b6ac-4b3d-aad0-4e97277dc85d"
-					(reference "#PWR0101")
+					(reference "#PWR0102")
 					(unit 1)
 				)
@@
 		(dnp no)
 		(fields_autoplaced yes)
-		(property "Reference" "#PWR0100"
+		(property "Reference" "#PWR0101"
 			(at 97.79 156.21 0)
 			(effects
@@
 			(project "linht-hw"
 				(path "/73efc1fc-21f6-4aef-9f73-508fe18fa32e/5f168690-b6ac-4b3d-aad0-4e97277dc85d"
-					(reference "#PWR0100")
+					(reference "#PWR0101")
 					(unit 1)
 				)

Commit message: minor power on/off circuit tweaks
Parts:
- renumbered D6 to D7, R45 to R46, R46 to R47, R47 to R48
Changed lines of the file:
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@@
 		(on_board yes)
 		(dnp no)
-		(property "Reference" "R45"
+		(property "Reference" "R46"
 			(at 59.69 138.43 90)
 			(effects
@@
 			(project "linht-hw"
 				(path "/73efc1fc-21f6-4aef-9f73-508fe18fa32e/5f168690-b6ac-4b3d-aad0-4e97277dc85d"
-					(reference "R45")
+					(reference "R46")
 					(unit 1)
 				)
@@
 		(on_board yes)
 		(dnp no)
-		(property "Reference" "R46"
+		(property "Reference" "R47"
 			(at 59.69 146.05 90)
 			(effects
@@
 			(project "linht-hw"
 				(path "/73efc1fc-21f6-4aef-9f73-508fe18fa32e/5f168690-b6ac-4b3d-aad0-4e97277dc85d"
-					(reference "R46")
+					(reference "R47")
 					(unit 1)
 				)
@@
 		(dnp no)
 		(fields_autoplaced yes)
-		(property "Reference" "D6"
+		(property "Reference" "D7"
 			(at 61.2775 129.54 0)
 			(effects
@@
 			(project "linht-hw"
 				(path "/73efc1fc-21f6-4aef-9f73-508fe18fa32e/5f168690-b6ac-4b3d-aad0-4e97277dc85d"
-					(reference "D6")
+					(reference "D7")
 					(unit 1)
 				)
@@
 		(on_board yes)
 		(dnp no)
-		(property "Reference" "R47"
+		(property "Reference" "R48"
 			(at 185.42 111.76 90)
 			(effects
@@
 			(project ""
 				(path "/73efc1fc-21f6-4aef-9f73-508fe18fa32e/5f168690-b6ac-4b3d-aad0-4e97277dc85d"
-					(reference "R47")
-					(unit 1)
-				)
+					(reference "R48")
+					(unit 1)
+				)

Commit message: Added modified footprint for the PJ-204 audio 2.5 mm jack
This alternative footprint does not have three mounting mechanical
holes. This will make the jack body 0.5 mm higher, making it better
aligned with the center of the 3.5 mm jack.
Parts:
- J13: footprint parts:Jack_2.5mm_PJ-204_Horizontal -> parts:Jack_2.5mm_PJ-204_nodrill_Horizontal
Changed lines of the file:
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@@
 			)
 		)
-		(property "Footprint" "parts:Jack_2.5mm_PJ-204_Horizontal"
+		(property "Footprint" "parts:Jack_2.5mm_PJ-204_nodrill_Horizontal"
 			(at 196.85 74.93 0)
 			(effects
