File: connectors.kicad_sch (KiCad schematic)
At the start: 19 parts, among them J12 USB_C, J13 2.5mm, J14 3.5mm, U8 USBLC6-2SC6

Commit message: Added on/off switch and volume pot to schematics and layout
Parts:
- added C60: 100n, Capacitor_SMD:C_0402_1005Metric, symbol Device:C_Small
- added R49: ?R, Resistor_SMD:R_0402_1005Metric, symbol Device:R_Small
- added SW2: 10k, parts:Connector_08x09mm_pot_switch, symbol parts:Potentiometer_Switch
Connections:
- net GND: now also C60.2, SW2.3, SW2.S2
- new net: R49.2, SW2.1
- new net +3V3: C60.1, R49.1
- new net SWITCH_ON_OFF: SW2.S1
- new net VOL_POT: SW2.2

Commit message: Fixed majority of ERC warnings and errors
Parts:
- J12: symbol Connector:USB_C_Receptacle_USB2.0 -> Connector:USB_C_Receptacle_USB2.0_16P
Changed lines of the file:
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@@
 			)
 		)
-		(property "Datasheet" ""
+		(property "Datasheet" "~"
 			(at 96.52 102.87 0)
 			(effects
@@
 			)
 		)
-		(property "Description" ""
+		(property "Description" "Resistor, small symbol"
 			(at 96.52 102.87 0)
 			(effects
@@
 			)
 		)
-		(property "Datasheet" ""
+		(property "Datasheet" "~"
 			(at 59.69 140.97 0)
 			(effects
@@
 			)
 		)
-		(property "Description" ""
+		(property "Description" "Resistor, small symbol"
 			(at 59.69 140.97 0)
 			(effects
@@
 			)
 		)
-		(property "Datasheet" ""
+		(property "Datasheet" "~"
 			(at 59.69 143.51 0)
 			(effects
@@
 			)
 		)
-		(property "Description" ""
+		(property "Description" "Resistor, small symbol"
 			(at 59.69 143.51 0)
 			(effects
@@
 			)
 		)
-		(property "Description" ""
+		(property "Description" "Power symbol creates a global label with name \"+3V3\""
 			(at 96.52 97.79 0)
 			(effects
@@
 	)
 	(symbol
-		(lib_id "Connector:USB_C_Receptacle_USB2.0")
+		(lib_id "Connector:USB_C_Receptacle_USB2.0_16P")
 		(at 39.37 151.13 0)
 		(unit 1)
@@
 			)
 		)
-		(property "Description" ""
+		(property "Description" "USB 2.0-only 16P Type-C Receptacle connector"
 			(at 39.37 151.13 0)
 			(effects

Commit message: Fixed minor schematic issues
Parts:
- added J3: GND spring, TestPoint:TestPoint_Pad_D4.0mm, symbol Connector_Generic:Conn_01x01
Connections:
- net GND: now also J3.1 (Pin_1)
- net USB_DN: now also U8.4 (I/O2); no longer U8.6 (I/O1)
- net USB_DP: now also U8.6 (I/O1); no longer U8.4 (I/O2)
- net xUDN: now also U8.3 (I/O2); no longer U8.1 (I/O1)
- net xUDP: now also U8.1 (I/O1); no longer U8.3 (I/O2)
Changed lines of the file:
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@@
+	(wire
+		(pts
+			(xy 132.08 62.23) (xy 129.54 62.23)
+		)
+		(stroke
+			(width 0)
+			(type default)
+		)
+	)
 	(wire
 		(pts
@@
 		(pts
 			(xy 73.66 165.1) (xy 81.28 165.1)
+		)
+		(stroke
+			(width 0)
+			(type default)
+		)
+	)
+	(wire
+		(pts
+			(xy 129.54 62.23) (xy 129.54 64.77)
 		)
 		(stroke
@@
 					(size 1.524 1.524)
 				)
+				(hide yes)
 			)
 		)
@@
 					(size 1.524 1.524)
 				)
+				(hide yes)
 			)
 		)
@@
 					(size 1.524 1.524)
 				)
+				(hide yes)
 			)
 		)
@@
 		(lib_id "Power_Protection:USBLC6-2SC6")
 		(at 83.82 153.67 270)
+		(mirror x)
 		(unit 1)
 		(exclude_from_sim no)
@@
 		(dnp no)
 		(property "Reference" "U8"
-			(at 83.82 167.005 90)
+			(at 83.82 169.037 90)
 			(effects
 				(font
@@
 		)
 		(property "Value" "USBLC6-2SC6"
-			(at 83.82 168.91 90)
+			(at 83.82 167.132 90)
 			(effects
 				(font
@@
 		)
 		(property "Datasheet" "https://www.st.com/resource/en/datasheet/usblc6-2.pdf"
-			(at 92.71 158.75 0)
+			(at 92.71 148.59 0)
 			(effects
 				(font
@@
 	(symbol
 		(lib_id "power:GND")
+		(at 129.54 64.77 0)
+		(mirror y)
+		(unit 1)
+		(exclude_from_sim no)
+		(in_bom yes)
+		(on_board yes)
+		(dnp no)
+		(property "Reference" "#PWR055"
+			(at 129.54 71.12 0)
+			(effects
+				(font
+					(size 1.27 1.27)
+				)
+				(hide yes)
+			)
+		)
+		(property "Value" "GND"
+			(at 129.54 69.85 0)
+			(effects
+				(font
+					(size 1.27 1.27)
+				)
+			)
+		)
+		(property "Footprint" ""
+			(at 129.54 64.77 0)
+			(effects
+				(font
+					(size 1.27 1.27)
+				)
+				(hide yes)
+			)
+		)
+		(property "Datasheet" ""
+			(at 129.54 64.77 0)
+			(effects
+				(font
+					(size 1.27 1.27)
+				)
+				(hide yes)
+			)
+		)
+		(property "Description" "Power symbol creates a global label with name \"GND\" , ground"
+			(at 129.54 64.77 0)
+			(effects
+				(font
+					(size 1.27 1.27)
+				)
+				(hide yes)
+			)
+		)
+		(pin "1"
+		)
+		(instances
+			(project "linht-hw"
+				(path "/73efc1fc-21f6-4aef-9f73-508fe18fa32e/5f168690-b6ac-4b3d-aad0-4e97277dc85d"
+					(reference "#PWR055")
+					(unit 1)
+				)
+			)
+		)
+	)
+	(symbol
+		(lib_id "power:GND")
 		(at 189.23 80.01 0)
 		(unit 1)
@@
 					(unit 1)
 				)
+			)
+		)
+	)
+	(symbol
+		(lib_id "Connector_Generic:Conn_01x01")
+		(at 137.16 62.23 0)
+		(mirror x)
+		(unit 1)
+		(exclude_from_sim no)
+		(in_bom yes)
+		(on_board yes)
+		(dnp no)
+		(fields_autoplaced yes)
+		(property "Reference" "J3"
+			(at 137.16 56.8155 0)
+			(effects
+				(font
+					(size 1.27 1.27)
+				)
+			)
+		)
+		(property "Value" "GND spring"
+			(at 137.16 59.2398 0)
+			(effects
+				(font
+					(size 1.27 1.27)
+				)
+			)
+		)
+		(property "Footprint" "TestPoint:TestPoint_Pad_D4.0mm"
+			(at 137.16 62.23 0)
+			(effects
+				(font
+					(size 1.27 1.27)
+				)
+				(hide yes)
+			)
+		)
+		(property "Datasheet" "~"
+			(at 137.16 62.23 0)
+			(effects
+				(font
+					(size 1.27 1.27)
+				)
+				(hide yes)
+			)
+		)
+		(property "Description" "Generic connector, single row, 01x01, script generated (kicad-library-utils/schlib/autogen/connector/)"
+			(at 137.16 62.23 0)
+			(effects
+				(font
+					(size 1.27 1.27)
+				)
+				(hide yes)
+			)
+		)
+		(pin "1"
+		)
+		(instances
+			(project "linht-hw"
+				(path "/73efc1fc-21f6-4aef-9f73-508fe18fa32e/5f168690-b6ac-4b3d-aad0-4e97277dc85d"
+					(reference "J3")
+					(unit 1)
+				)

Commit message: Changed resistor value for the volume to 15 kΩ
Parts:
- R49: value ?R -> 15k
Changed lines of the file:
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@@
 		(comment 1 "Author: Wojciech SP5WWP, Andy OE3ANC, Vlastimil OK5VAS")
 	)
-	(text_box "TODO: The value of the potentiometer is 10 kOhm. Set the value of the resistor above accordingly."
+	(text_box "ADC V_{ref} = 1.8 V\nWith 10 kΩ potentiometer and\n15 kΩ resistor this means a\nrange of 0-1.32 V."
 		(exclude_from_sim no)
-		(at 102.235 90.805 0)
-		(size 29.21 8.89)
+		(at 102.235 86.36 0)
+		(size 32.385 13.335)
 		(margins 0.9525 0.9525 0.9525 0.9525)
 		(stroke
@@
 				(size 1.27 1.27)
 			)
-			(justify left top)
+			(justify left)
 		)
 	)
@@
 			)
 		)
-		(property "Value" "?R"
+		(property "Value" "15k"
 			(at 93.472 103.886 0)
 			(effects
