File: display.kicad_sch (KiCad schematic)
At the start: 17 parts, among them J5 LCD, Q3 BSS138, Q4 BSS138

Commit message: Assigned footprint and set position on PCB for the LEDs
Parts:
- D4, D5: footprint (none) -> LED_SMD:LED_0402_1005Metric
- D6: footprint (none) -> LED_THT:LED_Rectangular_W3.0mm_H2.0mm
Changed lines of the file:
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@@
 			)
 		)
-		(property "Footprint" ""
+		(property "Footprint" "LED_THT:LED_Rectangular_W3.0mm_H2.0mm"
 			(at 209.55 90.17 0)
 			(effects
@@
 			)
 		)
-		(property "Footprint" ""
+		(property "Footprint" "LED_SMD:LED_0402_1005Metric"
 			(at 209.55 68.58 0)
 			(effects
@@
 			)
 		)
-		(property "Footprint" ""
+		(property "Footprint" "LED_SMD:LED_0402_1005Metric"
 			(at 209.55 80.01 0)
 			(effects

Commit message: New footprint for the 20 pin display connector
Parts:
- J5: footprint (none) -> parts:Connector_FFC_01x20_P0.75mm
Changed lines of the file:
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@@
 			)
 		)
-		(property "Footprint" ""
+		(property "Footprint" "parts:Connector_FFC_01x20_P0.75mm"
 			(at 119.38 85.09 0)
 			(effects

Commit message: Connected display pins 6-12 and 14 to the GND
Based on the original Retevis C62 PCB, these pins are grounded.
Connections:
- net GND: now also J5.10 (Pin_10), J5.11 (Pin_11), J5.12 (Pin_12), J5.14 (Pin_14), J5.6 (Pin_6), J5.7 (Pin_7), J5.8 (Pin_8), J5.9 (Pin_9)
- no-connect marks 8 -> 0
Changed lines of the file:
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@@
+	)
+	(junction
+		(at 110.49 90.17)
+		(diameter 0)
+		(color 0 0 0 0)
 	)
 	(junction
@@
 	)
 	(junction
+		(at 110.49 74.93)
+		(diameter 0)
+		(color 0 0 0 0)
+	)
+	(junction
+		(at 110.49 77.47)
+		(diameter 0)
+		(color 0 0 0 0)
+	)
+	(junction
 		(at 226.06 68.58)
+		(diameter 0)
+		(color 0 0 0 0)
+	)
+	(junction
+		(at 110.49 80.01)
 		(diameter 0)
 		(color 0 0 0 0)
@@
 	)
 	(junction
+		(at 110.49 82.55)
+		(diameter 0)
+		(color 0 0 0 0)
+	)
+	(junction
 		(at 96.52 64.77)
+		(diameter 0)
+		(color 0 0 0 0)
+	)
+	(junction
+		(at 110.49 85.09)
 		(diameter 0)
 		(color 0 0 0 0)
@@
 	)
 	(junction
+		(at 110.49 87.63)
+		(diameter 0)
+		(color 0 0 0 0)
+	)
+	(junction
 		(at 101.6 128.27)
 		(diameter 0)
 		(color 0 0 0 0)
 	)
-	(no_connect
-		(at 114.3 85.09)
-	)
-	(no_connect
-		(at 114.3 74.93)
-	)
-	(no_connect
-		(at 114.3 82.55)
-	)
-	(no_connect
-		(at 114.3 90.17)
-	)
-	(no_connect
-		(at 114.3 87.63)
-	)
-	(no_connect
-		(at 114.3 95.25)
-	)
-	(no_connect
-		(at 114.3 77.47)
-	)
-	(no_connect
-		(at 114.3 80.01)
-	)
 	(wire
 		(pts
@@
 	(wire
 		(pts
+			(xy 110.49 80.01) (xy 114.3 80.01)
+		)
+		(stroke
+			(width 0)
+			(type default)
+		)
+	)
+	(wire
+		(pts
+			(xy 110.49 95.25) (xy 110.49 90.17)
+		)
+		(stroke
+			(width 0)
+			(type default)
+		)
+	)
+	(wire
+		(pts
 			(xy 114.3 69.85) (xy 96.52 69.85)
 		)
@@
 	(wire
 		(pts
+			(xy 114.3 90.17) (xy 110.49 90.17)
+		)
+		(stroke
+			(width 0)
+			(type default)
+		)
+	)
+	(wire
+		(pts
 			(xy 189.23 99.06) (xy 191.77 99.06)
 		)
@@
 	(wire
 		(pts
+			(xy 110.49 85.09) (xy 114.3 85.09)
+		)
+		(stroke
+			(width 0)
+			(type default)
+		)
+	)
+	(wire
+		(pts
 			(xy 201.93 104.14) (xy 201.93 106.68)
 		)
@@
 	(wire
 		(pts
+			(xy 110.49 87.63) (xy 110.49 90.17)
+		)
+		(stroke
+			(width 0)
+			(type default)
+		)
+	)
+	(wire
+		(pts
 			(xy 191.77 99.06) (xy 194.31 99.06)
 		)
@@
 	(wire
 		(pts
+			(xy 110.49 77.47) (xy 114.3 77.47)
+		)
+		(stroke
+			(width 0)
+			(type default)
+		)
+	)
+	(wire
+		(pts
+			(xy 110.49 77.47) (xy 110.49 80.01)
+		)
+		(stroke
+			(width 0)
+			(type default)
+		)
+	)
+	(wire
+		(pts
 			(xy 93.98 105.41) (xy 114.3 105.41)
 		)
@@
 	(wire
 		(pts
+			(xy 110.49 87.63) (xy 114.3 87.63)
+		)
+		(stroke
+			(width 0)
+			(type default)
+		)
+	)
+	(wire
+		(pts
 			(xy 110.49 67.31) (xy 114.3 67.31)
 		)
@@
 	(wire
 		(pts
+			(xy 110.49 80.01) (xy 110.49 82.55)
+		)
+		(stroke
+			(width 0)
+			(type default)
+		)
+	)
+	(wire
+		(pts
 			(xy 110.49 62.23) (xy 114.3 62.23)
 		)
@@
 	(wire
 		(pts
+			(xy 110.49 82.55) (xy 110.49 85.09)
+		)
+		(stroke
+			(width 0)
+			(type default)
+		)
+	)
+	(wire
+		(pts
 			(xy 179.07 99.06) (xy 181.61 99.06)
 		)
@@
 	(wire
 		(pts
+			(xy 110.49 74.93) (xy 110.49 77.47)
+		)
+		(stroke
+			(width 0)
+			(type default)
+		)
+	)
+	(wire
+		(pts
 			(xy 101.6 102.87) (xy 101.6 86.36)
 		)
@@
 	(wire
 		(pts
+			(xy 110.49 74.93) (xy 114.3 74.93)
+		)
+		(stroke
+			(width 0)
+			(type default)
+		)
+	)
+	(wire
+		(pts
+			(xy 114.3 95.25) (xy 110.49 95.25)
+		)
+		(stroke
+			(width 0)
+			(type default)
+		)
+	)
+	(wire
+		(pts
 			(xy 226.06 90.17) (xy 226.06 80.01)
 		)
@@
 	(wire
 		(pts
+			(xy 97.79 90.17) (xy 110.49 90.17)
+		)
+		(stroke
+			(width 0)
+			(type default)
+		)
+	)
+	(wire
+		(pts
+			(xy 110.49 85.09) (xy 110.49 87.63)
+		)
+		(stroke
+			(width 0)
+			(type default)
+		)
+	)
+	(wire
+		(pts
+			(xy 110.49 67.31) (xy 110.49 74.93)
+		)
+		(stroke
+			(width 0)
+			(type default)
+		)
+	)
+	(wire
+		(pts
 			(xy 111.76 133.35) (xy 111.76 139.7)
 		)
@@
 	(wire
 		(pts
+			(xy 110.49 82.55) (xy 114.3 82.55)
+		)
+		(stroke
+			(width 0)
+			(type default)
+		)
+	)
+	(wire
+		(pts
 			(xy 114.3 107.95) (xy 107.95 107.95)
 		)
@@
 		(pts
 			(xy 96.52 69.85) (xy 96.52 64.77)
-		)
-		(stroke
-			(width 0)
-			(type default)
-		)
-	)
-	(wire
-		(pts
-			(xy 110.49 67.31) (xy 110.49 74.93)
 		)
 		(stroke
@@
 	(symbol
 		(lib_id "power:GND")
-		(at 110.49 74.93 0)
+		(at 97.79 90.17 270)
 		(unit 1)
 		(exclude_from_sim no)
@@
 		(fields_autoplaced yes)
 		(property "Reference" "#PWR085"
-			(at 110.49 81.28 0)
+			(at 91.44 90.17 0)
 			(effects
 				(font
@@
 		)
 		(property "Value" "GND"
-			(at 110.49 79.0631 0)
+			(at 96.52 86.36 90)
 			(effects
 				(font
@@
 		)
 		(property "Footprint" ""
-			(at 110.49 74.93 0)
+			(at 97.79 90.17 0)
 			(effects
 				(font
@@
 		)
 		(property "Datasheet" ""
-			(at 110.49 74.93 0)
+			(at 97.79 90.17 0)
 			(effects
 				(font
@@
 		)
 		(property "Description" "Power symbol creates a global label with name \"GND\" , ground"
-			(at 110.49 74.93 0)
-			(effects
-				(font
+			(at 97.79 90.17 0)
+			(effects
+				(font

Commit message: Fixed majority of ERC warnings and errors
Changed lines of the file:
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@@
 			)
 		)
-		(property "Description" ""
+		(property "Description" "Power symbol creates a global label with name \"+3V3\""
 			(at 96.52 60.96 0)
 			(effects

Commit message: Changed LED power from 5V to 3.3 V and fixed their resistor values
Parts:
- R40, R41: value 1k -> 220R
Connections:
- net +3V3: now also R40.2, R41.2
- net +5V: no longer R40.2, R41.2
Other:
- note removed: "TODO: Confirm resistor values"
Changed lines of the file:
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@@
-		)
-	)
-	(text "TODO: Confirm resistor values"
-		(exclude_from_sim no)
-		(at 242.57 73.66 0)
-		(effects
-			(font
-				(size 1.27 1.27)
-			)
 		)
 	)
@@
 	)
 	(junction
-		(at 226.06 80.01)
-		(diameter 0)
-		(color 0 0 0 0)
-	)
-	(junction
 		(at 110.49 87.63)
 		(diameter 0)
@@
 	(wire
 		(pts
+			(xy 226.06 88.9) (xy 226.06 90.17)
+		)
+		(stroke
+			(width 0)
+			(type default)
+		)
+	)
+	(wire
+		(pts
 			(xy 223.52 68.58) (xy 226.06 68.58)
 		)
@@
 		(pts
 			(xy 114.3 95.25) (xy 110.49 95.25)
-		)
-		(stroke
-			(width 0)
-			(type default)
-		)
-	)
-	(wire
-		(pts
-			(xy 226.06 90.17) (xy 226.06 80.01)
 		)
 		(stroke
@@
 			)
 		)
-		(property "Value" "1k"
+		(property "Value" "220R"
 			(at 219.71 71.3162 90)
 			(effects
@@
 	)
 	(symbol
+		(lib_id "power:+3V3")
+		(at 226.06 66.04 0)
+		(unit 1)
+		(exclude_from_sim no)
+		(in_bom yes)
+		(on_board yes)
+		(dnp no)
+		(fields_autoplaced yes)
+		(property "Reference" "#PWR034"
+			(at 226.06 69.85 0)
+			(effects
+				(font
+					(size 1.27 1.27)
+				)
+				(hide yes)
+			)
+		)
+		(property "Value" "+3V3"
+			(at 226.06 61.9069 0)
+			(effects
+				(font
+					(size 1.27 1.27)
+				)
+			)
+		)
+		(property "Footprint" ""
+			(at 226.06 66.04 0)
+			(effects
+				(font
+					(size 1.27 1.27)
+				)
+				(hide yes)
+			)
+		)
+		(property "Datasheet" ""
+			(at 226.06 66.04 0)
+			(effects
+				(font
+					(size 1.27 1.27)
+				)
+				(hide yes)
+			)
+		)
+		(property "Description" "Power symbol creates a global label with name \"+3V3\""
+			(at 226.06 66.04 0)
+			(effects
+				(font
+					(size 1.27 1.27)
+				)
+				(hide yes)
+			)
+		)
+		(pin "1"
+		)
+		(instances
+			(project "linht-hw"
+				(path "/73efc1fc-21f6-4aef-9f73-508fe18fa32e/42192b89-bd04-4531-bec0-520394b48a86"
+					(reference "#PWR034")
+					(unit 1)
+				)
+			)
+		)
+	)
+	(symbol
 		(lib_id "Device:R")
 		(at 101.6 82.55 180)
@@
 			)
 		)
-		(property "Value" "1k"
+		(property "Value" "220R"
 			(at 219.71 82.7462 90)
 			(effects
@@
 	(symbol
 		(lib_id "power:+5V")
-		(at 226.06 66.04 0)
+		(at 226.06 88.9 0)
 		(unit 1)
 		(exclude_from_sim no)
@@
 		(fields_autoplaced yes)
 		(property "Reference" "#PWR089"
-			(at 226.06 69.85 0)
+			(at 226.06 92.71 0)
 			(effects
 				(font
@@
 		)
 		(property "Value" "+5V"
-			(at 226.06 61.9069 0)
+			(at 226.06 84.7669 0)
 			(effects
 				(font
@@
 		)
 		(property "Footprint" ""
-			(at 226.06 66.04 0)
+			(at 226.06 88.9 0)
 			(effects
 				(font
@@
 		)
 		(property "Datasheet" ""
-			(at 226.06 66.04 0)
+			(at 226.06 88.9 0)
 			(effects
 				(font
@@
 		)
 		(property "Description" "Power symbol creates a global label with name \"+5V\""
-			(at 226.06 66.04 0)
-			(effects
-				(font
+			(at 226.06 88.9 0)
+			(effects
+				(font
