File: power.kicad_sch (KiCad schematic)
At the start: 28 parts, among them J2 Battery connector, U5 TPS562203, U7 TPS562203

Commit message: updates
- updated the 5V line (diode connected sources - USB and DC/DC)
- proposed a power on-off circuit based on a XNOR gate
- reannotated the schematic
- updated the PDF
Parts:
- added C21: 100n, Capacitor_SMD:C_0402_1005Metric, symbol Device:C
- added C22: 10u, Capacitor_SMD:C_1206_3216Metric, symbol Device:C
- added D1: BAT60A, Diode_SMD:D_SOD-323, symbol Diode:BAT60A
- added Q1: BSS138, Package_TO_SOT_SMD:SOT-23, symbol Transistor_FET:BSS138
- added R17, R23: 47k, Resistor_SMD:R_0402_1005Metric, symbol Device:R
- added R18: 100k, Resistor_SMD:R_0402_1005Metric, symbol Device:R
- added SW1: SW_SPST, symbol Switch:SW_SPST
- added U5: 74AHC1G86, symbol 74xGxx:74AHC1G86
- renumbered C40 to C16, C42 to C17, C16 to C18, C39 to C19, C43 to C20, C35 to C23, C26 to C24, C41 to C25, C51 to C26, C36 to C27, C52 to C28, C37 to C29, C53 to C30, C38 to C31, C54 to C32, R39 to R15, R42 to R16, R37 to R19, R38 to R20, R43 to R21, R45 to R22, U5 to U3, U7 to U4
Connections:
- net +3V3: now also C21.1, R17.1, R23.1, U5.5 (VCC)
- net +5V: now also D1.1 (K); no longer C25.1, C27.1, C29.1, C31.1, L3.2, R19.1
- net GND: now also C21.2, C22.2, Q1.2 (S), SW1.1 (A), U5.3 (GND)
- new net: C22.1, R18.2, U5.2
- new net: C25.1, C27.1, C29.1, C31.1, D1.2 (A), L3.2, R19.1
- new net: Q1.1 (G), U5.4
- new net ON/OFF: Q1.3 (D), R23.2
- new net PWR_SW: R17.2, R18.1, SW1.2 (B), U5.1
Other:
- moved on the sheet: C16, C17, C18, C19, C20, C23, C24, C25, C26, C27, C28, C29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

Commit message: tweaked the power-on circuit
- supplied the XNOR gate with 5V instead of 3.3V
- added a MOSFET to drive the 3.3V DC/DC converter's EN pin
- removed a pull-up resistor at the ON/OFF line
Parts:
- removed R23: 47k, Resistor_SMD:R_0402_1005Metric, symbol Device:R
- added C16: 10u, Capacitor_SMD:C_1206_3216Metric, symbol Device:C
- added D1: BAT60A, Diode_SMD:D_SOD-323, symbol Diode:BAT60A
- added Q1: BSS138, Package_TO_SOT_SMD:SOT-23, symbol Transistor_FET:BSS138
- added R13: 100R, Resistor_SMD:R_0402_1005Metric, symbol Device:R
- renumbered C16 to C17, C17 to C18, C18 to C19, C19 to C20, C20 to C21, C21 to C22, C22 to C23, C23 to C24, C24 to C25, C25 to C26, C26 to C27, C27 to C28, C28 to C29, C29 to C30, C30 to C31, C31 to C32, C32 to C33, D1 to D2, Q1 to Q2, R13 to R14, R14 to R15, R15 to R16, R16 to R17, R17 to R18, R18 to R19, R19 to R20, R20 to R21, R21 to R22, R22 to R23
Connections:
- net +3V3: no longer C22.1, R18.1, U5.5 (VCC)
- net +5V: now also C22.1, R18.1, U5.5 (VCC)
- net GND: now also C16.2, Q1.2 (S)
- net PWR_SW: now also D1.2 (A); no longer R18.2, R19.1, SW1.2 (B), U5.1
- net 3V3_EN: now reaches R17.2, U4.5 (EN)
- net 3V3_EN: now also C16.1, R13.1
- new net: Q1.1 (G), R18.2, R19.1, SW1.2 (B), U5.1
- new net: D1.1 (K), Q1.3 (D), R13.2

Commit message: minor power on/off circuit tweaks
Parts:
- added D2: BAT60A, Diode_SMD:D_SOD-323, symbol Diode:BAT60A
- added R20: 100k, Resistor_SMD:R_0402_1005Metric, symbol Device:R
- R16: renamed from R18; value 47k -> 51k
- renumbered C23 to C22, C24 to C23, C25 to C24, C22 to C25, D2 to D3, R16 to R17, R17 to R18, R20 to R21, R21 to R22, R22 to R23, R23 to R24
Connections:
- net at Q1.1 (G), R16.2, R19.1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: now also R20.1
- net at C22.1, U5.2: now also D2.1 (K), R20.2; no longer R19.2
- new net: D2.2 (A), R19.2
Other:
- note added: "Power switch (volume knob)"
- moved on the sheet: C16, C17, C18, C19, C20, C21, C22, C23, C24, C25, C26, C27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

Commit message: Assigned footprint and layout position of the battery connector
Parts:
- J2: footprint (none) -> parts:Connector_01x03_BT-003E
Changed lines of the file:
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@@
 			)
 		)
-		(property "Footprint" ""
+		(property "Footprint" "parts:Connector_01x03_BT-003E"
 			(at 49.53 55.88 0)
 			(effects
