File: power.kicad_sch (KiCad schematic)
At the start: 42 parts, among them J2 Battery connector, Q1 BSS138, Q2 BSS138, SW1 SW_SPST, U3 TPS562203, U4 TPS562203, U5 74AHC1G86

Commit message: Added on/off switch and volume pot to schematics and layout
Parts:
- removed SW1: SW_SPST, symbol Switch:SW_SPST
Connections:
- net SWITCH_ON_OFF: now reaches Q1.1 (G), R16.2, R19.1, R20.1, U5.1
Other:
- note removed: "Power switch (volume knob)"
Changed lines of the file:
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@@
 		)
 	)
-	(text "Power switch\n(volume knob)"
-		(exclude_from_sim no)
-		(at 66.04 184.15 0)
-		(effects
-			(font
-				(size 1.27 1.27)
-			)
-			(justify right)
-		)
-	)
 	(text "V_{FB} = 600 mV"
 		(exclude_from_sim no)
@@
 	(wire
 		(pts
-			(xy 97.79 173.99) (xy 109.22 173.99)
+			(xy 59.69 179.07) (xy 69.85 179.07)
 		)
 		(stroke
@@
 	(wire
 		(pts
-			(xy 207.01 53.34) (xy 207.01 52.07)
+			(xy 97.79 173.99) (xy 109.22 173.99)
 		)
 		(stroke
@@
 	(wire
 		(pts
-			(xy 125.73 55.88) (xy 123.19 55.88)
+			(xy 207.01 53.34) (xy 207.01 52.07)
 		)
 		(stroke
@@
 	(wire
 		(pts
-			(xy 63.5 115.57) (xy 63.5 116.84)
+			(xy 125.73 55.88) (xy 123.19 55.88)
 		)
 		(stroke
@@
 	(wire
 		(pts
-			(xy 57.15 58.42) (xy 57.15 59.69)
+			(xy 63.5 115.57) (xy 63.5 116.84)
 		)
 		(stroke
@@
 		)
 	)
-	(polyline
+	(wire
 		(pts
-			(xy 64.77 171.45) (xy 64.77 181.61)
+			(xy 57.15 58.42) (xy 57.15 59.69)
 		)
 		(stroke
@@
 	(wire
 		(pts
-			(xy 69.85 165.1) (xy 69.85 166.37)
+			(xy 214.63 53.34) (xy 207.01 53.34)
 		)
 		(stroke
@@
 	(wire
 		(pts
-			(xy 214.63 53.34) (xy 207.01 53.34)
+			(xy 157.48 104.14) (xy 157.48 106.68)
 		)
 		(stroke
@@
 	(wire
 		(pts
-			(xy 157.48 104.14) (xy 157.48 106.68)
+			(xy 101.6 105.41) (xy 101.6 99.06)
 		)
 		(stroke
@@
 	(wire
 		(pts
-			(xy 101.6 105.41) (xy 101.6 99.06)
+			(xy 69.85 165.1) (xy 69.85 179.07)
 		)
 		(stroke
@@
 		)
 	)
-	(polyline
-		(pts
-			(xy 67.31 171.45) (xy 64.77 171.45)
-		)
-		(stroke
-			(width 0)
-			(type default)
-		)
-	)
 	(wire
 		(pts
@@
 		)
 	)
+	(hierarchical_label "SWITCH_ON_OFF"
+		(shape input)
+		(at 59.69 179.07 180)
+		(effects
+			(font
+				(size 1.27 1.27)
+			)
+			(justify right)
+		)
+	)
 	(hierarchical_label "ON{slash}OFF"
 		(shape output)
@@
 	)
 	(symbol
-		(lib_id "Switch:SW_SPST")
-		(at 69.85 171.45 270)
-		(mirror x)
-		(unit 1)
-		(exclude_from_sim no)
-		(in_bom yes)
-		(on_board yes)
-		(dnp no)
-		(property "Reference" "SW1"
-			(at 74.93 173.99 90)
-			(effects
-				(font
-					(size 1.27 1.27)
-				)
-				(justify right)
-			)
-		)
-		(property "Value" "SW_SPST"
-			(at 68.707 172.6621 90)
-			(effects
-				(font
-					(size 1.27 1.27)
-				)
-				(justify right)
-				(hide yes)
-			)
-		)
-		(property "Footprint" ""
-			(at 69.85 171.45 0)
-			(effects
-				(font
-					(size 1.27 1.27)
-				)
-				(hide yes)
-			)
-		)
-		(property "Datasheet" "~"
-			(at 69.85 171.45 0)
-			(effects
-				(font
-					(size 1.27 1.27)
-				)
-				(hide yes)
-			)
-		)
-		(property "Description" "Single Pole Single Throw (SPST) switch"
-			(at 69.85 171.45 0)
-			(effects
-				(font
-					(size 1.27 1.27)
-				)
-				(hide yes)
-			)
-		)
-		(pin "1"
-		)
-		(pin "2"
-		)
-		(instances
-			(project ""
-				(path "/73efc1fc-21f6-4aef-9f73-508fe18fa32e/be402a1e-34f3-489f-9745-963b98ced0ff"
-					(reference "SW1")
-					(unit 1)
-				)
-			)
-		)
-	)
-	(symbol
 		(lib_id "power:PWR_FLAG")
 		(at 207.01 52.07 0)
@@
 					(unit 1)
 				)
-			)
-		)
-	)
-	(symbol
-		(lib_id "power:GND")
-		(at 69.85 176.53 0)
-		(unit 1)
-		(exclude_from_sim no)
-		(in_bom yes)
-		(on_board yes)
-		(dnp no)
-		(fields_autoplaced yes)
-		(property "Reference" "#PWR034"
-			(at 69.85 182.88 0)
-			(effects
-				(font
-					(size 1.27 1.27)
-				)
-				(hide yes)
-			)
-		)
-		(property "Value" "GND"
-			(at 69.85 180.6631 0)
-			(effects
-				(font
-					(size 1.27 1.27)
-				)
-			)
-		)
-		(property "Footprint" ""
-			(at 69.85 176.53 0)
-			(effects
-				(font
-					(size 1.27 1.27)
-				)
-				(hide yes)
-			)
-		)
-		(property "Datasheet" ""
-			(at 69.85 176.53 0)
-			(effects
-				(font
-					(size 1.27 1.27)
-				)
-				(hide yes)
-			)
-		)
-		(property "Description" "Power symbol creates a global label with name \"GND\" , ground"
-			(at 69.85 176.53 0)
-			(effects
-				(font
-					(size 1.27 1.27)
-				)
-				(hide yes)
-			)
-		)
-		(pin "1"
-		)
-		(instances
-			(project "linht-hw"
-				(path "/73efc1fc-21f6-4aef-9f73-508fe18fa32e/be402a1e-34f3-489f-9745-963b98ced0ff"
-					(reference "#PWR034")
-					(unit 1)
-				)

Commit message: Assigned missing footprints
Parts:
- U5: footprint (none) -> Package_TO_SOT_SMD:SOT-353_SC-70-5
Changed lines of the file:
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@@
 			)
 		)
-		(property "Footprint" ""
+		(property "Footprint" "Package_TO_SOT_SMD:SOT-353_SC-70-5"
 			(at 133.35 162.56 0)
 			(effects

Commit message: Fixed majority of ERC warnings and errors
Changed lines of the file:
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@@
 	)
 	(junction
+		(at 191.77 64.77)
+		(diameter 0)
+		(color 0 0 0 0)
+	)
+	(junction
 		(at 207.01 53.34)
 		(diameter 0)
@@
 	(wire
 		(pts
+			(xy 191.77 67.31) (xy 191.77 64.77)
+		)
+		(stroke
+			(width 0)
+			(type default)
+		)
+	)
+	(wire
+		(pts
 			(xy 201.93 53.34) (xy 207.01 53.34)
 		)
@@
 	)
 	(symbol
+		(lib_id "power:PWR_FLAG")
+		(at 191.77 67.31 180)
+		(unit 1)
+		(exclude_from_sim no)
+		(in_bom yes)
+		(on_board yes)
+		(dnp no)
+		(property "Reference" "#FLG06"
+			(at 191.77 69.215 0)
+			(effects
+				(font
+					(size 1.27 1.27)
+				)
+				(hide yes)
+			)
+		)
+		(property "Value" "PWR_FLAG"
+			(at 191.77 71.374 0)
+			(effects
+				(font
+					(size 1.27 1.27)
+				)
+			)
+		)
+		(property "Footprint" ""
+			(at 191.77 67.31 0)
+			(effects
+				(font
+					(size 1.27 1.27)
+				)
+				(hide yes)
+			)
+		)
+		(property "Datasheet" "~"
+			(at 191.77 67.31 0)
+			(effects
+				(font
+					(size 1.27 1.27)
+				)
+				(hide yes)
+			)
+		)
+		(property "Description" "Special symbol for telling ERC where power comes from"
+			(at 191.77 67.31 0)
+			(effects
+				(font
+					(size 1.27 1.27)
+				)
+				(hide yes)
+			)
+		)
+		(pin "1"
+		)
+		(instances
+			(project "linht-hw"
+				(path "/73efc1fc-21f6-4aef-9f73-508fe18fa32e/be402a1e-34f3-489f-9745-963b98ced0ff"
+					(reference "#FLG06")
+					(unit 1)
+				)
+			)
+		)
+	)
+	(symbol
 		(lib_id "Device:C")
 		(at 130.81 97.79 90)
@@
 	)
 	(symbol
-		(lib_name "BSS138_1")
 		(lib_id "Transistor_FET:BSS138")
 		(at 53.34 165.1 0)

Commit message: Changed footprint of the C16 capacitor from 1206 to 0402
Parts:
- C16: footprint Capacitor_SMD:C_1206_3216Metric -> Capacitor_SMD:C_0402_1005Metric
Changed lines of the file:
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@@
 			)
 		)
-		(property "Footprint" "Capacitor_SMD:C_1206_3216Metric"
+		(property "Footprint" "Capacitor_SMD:C_0402_1005Metric"
 			(at 39.0652 161.29 0)
 			(effects
