File: power.kicad_sch (KiCad schematic)
At the start: 72 parts, among them J2 2S Battery, Q6 BSS84, U12 BQ25792RQMR, U3 TPS562203, U4 TPS562203, U6 TLV74018PDBVR

Commit message: Removed battery voltage divider and `U_BATT_MON` signal to SoM
Battery voltage can and will be measured by the BQ25792RQ IC via I2C
register.
Parts:
- removed C19: 100n, Capacitor_SMD:C_0402_1005Metric, symbol Device:C
- removed R14: 39k/1%, Resistor_SMD:R_0402_1005Metric, symbol Device:R
- removed R15: 10k/1%, Resistor_SMD:R_0402_1005Metric, symbol Device:R
- removed TP7: BQ_TS, TestPoint:TestPoint_Pad_D1.0mm, symbol Connector:TestPoint_Alt
- removed TP8: BQ_GND, TestPoint:TestPoint_Pad_D1.0mm, symbol Connector:TestPoint_Alt
Other:
- moved on the sheet: C17, C18, C20, C21, C23, C24, C26, C27, C28, C29, C30, C31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

Commit message: Added power management ATTiny826
Fixes #32
Fixes #35
Fixes #23
Parts:
- removed D3: BZX84Cxx, Package_TO_SOT_SMD:SOT-23, symbol Diode:BZX84Cxx
- removed D9: RB751S40, Diode_SMD:D_SOD-523, symbol Device:D_Schottky
- removed Q6: BSS84, Package_TO_SOT_SMD:SOT-23, symbol Transistor_FET:BSS84
- removed R17, R71, R72: 100k, Resistor_SMD:R_0402_1005Metric, symbol Device:R
- added C16, C19: 2u2, Capacitor_SMD:C_0402_1005Metric, symbol Device:C
- added C22: 100n, Capacitor_SMD:C_0402_1005Metric, symbol Device:C
- added R13: 100k, Resistor_SMD:R_0402_1005Metric, symbol Device:R
- added R14: 1k, Resistor_SMD:R_0402_1005Metric, symbol Device:R_Small
- added TP10: UPDI_TX, TestPoint:TestPoint_Pad_D1.0mm, symbol Connector:TestPoint_Alt
- added TP11: UPDI_GND, TestPoint:TestPoint_Pad_D1.0mm, symbol Connector:TestPoint_Alt
- added TP7: UPDI_RX, TestPoint:TestPoint_Pad_D1.0mm, symbol Connector:TestPoint_Alt
- added TP8: PM_TX, TestPoint:TestPoint_Pad_D1.0mm, symbol Connector:TestPoint_Alt
- added TP9: PM_RX, TestPoint:TestPoint_Pad_D1.0mm, symbol Connector:TestPoint_Alt
- added U14: ATtiny826, Package_DFN_QFN:VQFN-20-1EP_3x3mm_P0.4mm_EP1.7x1.7mm, symbol MCU_Microchip_ATtiny:ATtiny826-M
- added U5: MCP1703Ax-330xxTT, Package_TO_SOT_SMD:SOT-23, symbol Regulator_Linear:MCP1703Ax-330xxTT
- U12: MPN 595-BQ25792RQMR -> BQ25792RQMR; PN BQ25792RQMR -> 595-BQ25792RQMR
Connections:
- net +BATT: now also C16.1, U5.3 (VI)
- net 3V3_ON_REQ: now also U14.8 (PA7)
- net GND: now also C16.2, C19.2, C22.2, R13.2, TP11.1, U14.21 (GND), U14.3 (GND), U5.1 (GND)
- net SCL: now also U14.14 (PB0)
- net SDA: now also U14.13 (PB1)
- net ~{5V_OFF_REQ}: now also U14.20 (PA1); no longer U3.5 (EN)
- net ~{5V_ON_OUT}: now also U14.1 (PA2)
- net ~{5V_ON_REQ}: now also U14.6 (PA5)
- new net: R14.2, TP7.1, U14.19 (~{RESET}/PA0)
- new net: TP9.1, U14.11 (PB3)
- new net: R14.1, TP10.1
- new net: TP8.1, U14.12 (PB2)
- new net +3.3VP: C19.1, C22.1, U14.4 (VCC), U5.2 (VO)
- new net 5V0_ON_REQ: R13.1, U14.7 (PA6), U3.5 (EN)
- new net SIDE_BTN: U14.9 (PB5)
- new net USB_BOOT: U14.2 (PA3)
- no-connect marks 1 -> 7
Other:
- note added: "2x DC/DC enable pin"
- note added: "Enable bootloader"
- note added: "ON/OFF SoM"
- note added: "ON/OFF Switch"
- note added: "PMIC_STBY_REQ"
- note added: "Power Management MCU"
- note added: "Programming, UART"
- moved on the sheet: C17, C18, C20, C21, C23, C24, C26, C27, C28, C29, C30, C31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

Commit message: Changed 5V DC/DC buck to TPS565242
Original buck has 2 A maximum current output. New one has up to 5 A.
Our design needs ~3 A maximum current.

Fixes #38
Parts:
- removed C23: 100n, Capacitor_SMD:C_0402_1005Metric, symbol Device:C
- L3: value 4.7 uH -> 2.2 uH; footprint Inductor_SMD:L_Bourns-SRN6028 -> parts:L_TDK_SPM6530; LCSC C3221249 -> C76855; MPN SRN6028-4R7M -> SPM6530T-2R2M; PN 652-SRN6028-4R7M -> 652-SPM6530T-2R2M
- U3: value TPS562203 -> TPS565242; symbol Regulator_Switching:TPS562203 -> parts:TPS565242; LCSC C22445511 -> C5219270; MPN TPS562203DRLR -> TPS565242DRLR; PN 595-TPS562203DRLR -> 595-TPS565242DRLR
Connections:
- net GND: now also U3.4 (AGND)
Changed lines of the file:
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@@
 		)
 	)
-	(text_box "Inductor FNR6028S4R7MT\n  I_{SAT} = 3.0 A\n  R_{DC} = 39 mOhm\n  f_{res} = 35 MHz\n  η = 95.8 %\n\nInductor SRN6028-4R7M\n  I_{SAT} = 2.8 A\n  R_{DC} = 38 mOhm\n  f_{res} = 34 MHz\n  η = 95.7 %"
+	(text_box "Inductor SPM6530T-2R2M\n  I_{SAT} = 8.4 A\n  R_{DC} = 17.3 mOhm\n  f_{res} > 10 MHz\n\nInductor SRN6028-4R7M\n  I_{SAT} = 2.8 A\n  R_{DC} = 38 mOhm\n  f_{res} = 34 MHz\n  η = 95.7 %"
 		(exclude_from_sim no)
 		(at 224.79 15.24 0)
@@
 		)
 	)
-	(text_box "Expected Parameters:\n  V_{in} = 6.0 - 8.4 V\n  V_{out} = 5 V ± 3.3%\n  I_{out} = 2 A\n  η = 93.7 %\n  Duty = 62 %\n  f_{SW} = 547 kHz"
+	(text_box "Expected Parameters:\n  V_{in} = 6.0 - 8.4 V\n  V_{out} = 5 V ± 3.6 %\n  I_{out} = 4 A\n  η = 94.8 %\n  Duty = 61 %\n  f_{SW} = 519 kHz"
 		(exclude_from_sim no)
 		(at 255.27 24.13 0)
@@
 	)
 	(junction
-		(at 220.98 48.26)
-		(diameter 0)
-		(color 0 0 0 0)
-	)
-	(junction
 		(at 130.81 33.02)
 		(diameter 0)
@@
 	)
 	(junction
+		(at 196.85 59.69)
+		(diameter 0)
+		(color 0 0 0 0)
+	)
+	(junction
 		(at 264.16 153.67)
 		(diameter 0)
@@
 	(wire
 		(pts
+			(xy 196.85 59.69) (xy 195.58 59.69)
+		)
+		(stroke
+			(width 0)
+			(type default)
+		)
+	)
+	(wire
+		(pts
 			(xy 147.32 48.26) (xy 172.72 48.26)
 		)
@@
 	(wire
 		(pts
+			(xy 195.58 59.69) (xy 195.58 58.42)
+		)
+		(stroke
+			(width 0)
+			(type default)
+		)
+	)
+	(wire
+		(pts
 			(xy 111.76 78.74) (xy 111.76 80.01)
 		)
@@
 	(wire
 		(pts
-			(xy 209.55 50.8) (xy 207.01 50.8)
-		)
-		(stroke
-			(width 0)
-			(type default)
-		)
-	)
-	(wire
-		(pts
 			(xy 62.23 19.05) (xy 73.66 19.05)
 		)
@@
 	(wire
 		(pts
+			(xy 198.12 59.69) (xy 196.85 59.69)
+		)
+		(stroke
+			(width 0)
+			(type default)
+		)
+	)
+	(wire
+		(pts
 			(xy 207.01 53.34) (xy 208.28 53.34)
 		)
@@
 	(wire
 		(pts
+			(xy 198.12 58.42) (xy 198.12 59.69)
+		)
+		(stroke
+			(width 0)
+			(type default)
+		)
+	)
+	(wire
+		(pts
 			(xy 231.14 60.96) (xy 231.14 63.5)
 		)
@@
 	(wire
 		(pts
-			(xy 220.98 48.26) (xy 222.25 48.26)
-		)
-		(stroke
-			(width 0)
-			(type default)
-		)
-	)
-	(wire
-		(pts
 			(xy 128.27 74.93) (xy 128.27 73.66)
 		)
@@
 	(wire
 		(pts
-			(xy 220.98 48.26) (xy 220.98 52.07)
-		)
-		(stroke
-			(width 0)
-			(type default)
-		)
-	)
-	(wire
-		(pts
 			(xy 260.35 143.51) (xy 264.16 143.51)
 		)
@@
 	(wire
 		(pts
-			(xy 209.55 52.07) (xy 209.55 50.8)
-		)
-		(stroke
-			(width 0)
-			(type default)
-		)
-	)
-	(wire
-		(pts
 			(xy 200.66 151.13) (xy 200.66 153.67)
 		)
@@
 	(wire
 		(pts
-			(xy 196.85 58.42) (xy 196.85 59.69)
+			(xy 196.85 59.69) (xy 196.85 60.96)
 		)
 		(stroke
@@
 	(wire
 		(pts
-			(xy 209.55 52.07) (xy 210.82 52.07)
-		)
-		(stroke
-			(width 0)
-			(type default)
-		)
-	)
-	(wire
-		(pts
 			(xy 275.59 88.9) (xy 275.59 91.44)
 		)
@@
 	(wire
 		(pts
-			(xy 220.98 52.07) (xy 218.44 52.07)
-		)
-		(stroke
-			(width 0)
-			(type default)
-		)
-	)
-	(wire
-		(pts
 			(xy 241.3 48.26) (xy 252.73 48.26)
 		)
@@
 	(wire
 		(pts
-			(xy 207.01 48.26) (xy 220.98 48.26)
+			(xy 207.01 48.26) (xy 222.25 48.26)
 		)
 		(stroke
@@
 	(symbol
 		(lib_id "Device:C")
-		(at 214.63 52.07 90)
-		(unit 1)
-		(exclude_from_sim no)
-		(in_bom yes)
-		(on_board yes)
-		(dnp no)
-		(property "Reference" "C23"
-			(at 214.63 56.388 90)
-			(effects
-				(font
-					(size 1.27 1.27)
-				)
-			)
-		)
-		(property "Value" "100n"
-			(at 214.63 58.928 90)
-			(effects
-				(font
-					(size 1.27 1.27)
-				)
-			)
-		)
-		(property "Footprint" "Capacitor_SMD:C_0402_1005Metric"
-			(at 218.44 51.1048 0)
-			(effects
-				(font
-					(size 1.27 1.27)
-				)
-				(hide yes)
-			)
-		)
-		(property "Datasheet" "~"
-			(at 214.63 52.07 0)
-			(effects
-				(font
-					(size 1.27 1.27)
-				)
-				(hide yes)
-			)
-		)
-		(property "Description" "Unpolarized capacitor"
-			(at 214.63 52.07 0)
-			(effects
-				(font
-					(size 1.27 1.27)
-				)
-				(hide yes)
-			)
-		)
-		(property "LCSC" "C1525"
-			(at 214.63 52.07 90)
-			(effects
-				(font
-					(size 1.27 1.27)
-				)
-				(hide yes)
-			)
-		)
-		(property "MPN" "CL05B104KO5NNNC"
-			(at 214.63 52.07 90)
-			(effects
-				(font
-					(size 1.27 1.27)
-				)
-				(hide yes)
-			)
-		)
-		(property "PN" " 187-CL05B104KO5NNNC "
-			(at 214.63 52.07 90)
-			(effects
-				(font
-					(size 1.27 1.27)
-				)
-				(hide yes)
-			)
-		)
-		(property "LCSC Part" ""
-			(at 214.63 52.07 90)
-			(effects
-				(font
-					(size 1.27 1.27)
-				)
-				(hide yes)
-			)
-		)
-		(pin "1"
-		)
-		(pin "2"
-		)
-		(instances
-			(project ""
-				(path "/73efc1fc-21f6-4aef-9f73-508fe18fa32e/be402a1e-34f3-489f-9745-963b98ced0ff"
-					(reference "C23")
-					(unit 1)
-				)
-			)
-		)
-	)
-	(symbol
-		(lib_id "Device:C")
 		(at 85.09 26.67 0)
 		(unit 1)
@@
 	(symbol
 		(lib_id "power:GND")
-		(at 196.85 59.69 0)
+		(at 196.85 60.96 0)
 		(unit 1)
 		(exclude_from_sim no)
@@
 		(fields_autoplaced yes)
 		(property "Reference" "#PWR040"
-			(at 196.85 66.04 0)
+			(at 196.85 67.31 0)
 			(effects
 				(font
@@
 		)
 		(property "Value" "GND"
-			(at 196.85 63.8231 0)
+			(at 196.85 65.0931 0)
 			(effects
 				(font
@@
 		)
 		(property "Footprint" ""
-			(at 196.85 59.69 0)
+			(at 196.85 60.96 0)
 			(effects
 				(font
@@
 		)
 		(property "Datasheet" ""
-			(at 196.85 59.69 0)
+			(at 196.85 60.96 0)
 			(effects
 				(font
@@
 		)
 		(property "Description" "Power symbol creates a global label with name \"GND\" , ground"
-			(at 196.85 59.69 0)
+			(at 196.85 60.96 0)
 			(effects
 				(font
@@
 	)
 	(symbol
-		(lib_id "Regulator_Switching:TPS562203")
+		(lib_id "parts:TPS565242")
 		(at 196.85 50.8 0)
 		(unit 1)
@@
 			)
 		)
-		(property "Value" "TPS562203"
+		(property "Value" "TPS565242"
 			(at 196.85 43.18 0)
 			(effects
@@
 			)
 		)
-		(property "Datasheet" "https://www.ti.com/lit/ds/symlink/tps562203.pdf"
+		(property "Datasheet" "https://www.ti.com/lit/ds/symlink/tps565242.pdf"
 			(at 196.85 50.8 0)
 			(effects
@@
 			)
 		)
-		(property "Description" "2A Synchronous Step-Down Voltage Regulator 600kHz, Adjustable Output Voltage, 4.5-17V Input Voltage, 0.6V-7V Output Voltage, SOT-563"
+		(property "Description" "A 5A synchronous step-down converter in SOT-563 package with an input voltage range of 3V to 16V."
 			(at 196.85 50.8 0)
 			(effects
@@
 			)
 		)
-		(property "LCSC" "C22445511"
+		(property "LCSC" "C5219270"
 			(at 196.85 50.8 0)
 			(effects
@@
 			)
 		)
-		(property "MPN" "TPS562203DRLR "
+		(property "MPN" "TPS565242DRLR"
 			(at 196.85 50.8 0)
 			(effects
@@
 			)
 		)
-		(property "PN" "595-TPS562203DRLR "
+		(property "PN" "595-TPS565242DRLR"
 			(at 196.85 50.8 0)
 			(effects
@@
 			)
 		)
-		(property "Value" "4.7 uH"
+		(property "Value" "2.2 uH"
 			(at 226.06 45.72 90)
 			(effects
@@
 			)
 		)
-		(property "Footprint" "Inductor_SMD:L_Bourns-SRN6028"
+		(property "Footprint" "parts:L_TDK_SPM6530"
 			(at 226.06 48.26 0)
 			(effects
@@
 			)
 		)
-		(property "LCSC" "C3221249"
+		(property "LCSC" "C76855"
 			(at 226.06 48.26 90)
 			(effects
@@
 			)
 		)
-		(property "MPN" " SRN6028-4R7M "
+		(property "MPN" "SPM6530T-2R2M"
 			(at 226.06 48.26 90)
 			(effects
@@
 			)
 		)
-		(property "PN" "652-SRN6028-4R7M "
+		(property "PN" "652-SPM6530T-2R2M"
 			(at 226.06 48.26 90)
 			(effects

Commit message: Minor schematics tweaks and pinout optimizations
Connections:
- net ~{5V_ON_OUT}: now also U14.6 (PA5); no longer U14.1 (PA2)
- net ~{5V_ON_REQ}: now also U14.1 (PA2); no longer U14.6 (PA5)
- net SOM_RST: now reaches U14.5 (PA4)
- no-connect marks 7 -> 6
Changed lines of the file:
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@@
 	(text "ON/OFF Switch"
 		(exclude_from_sim no)
-		(at 119.634 161.544 0)
+		(at 119.634 153.924 0)
 		(effects
 			(font
@@
 	(text "ON/OFF SoM"
 		(exclude_from_sim no)
-		(at 119.634 153.924 0)
+		(at 119.634 161.544 0)
 		(effects
 			(font
@@
 	)
 	(no_connect
-		(at 93.98 158.75)
-	)
-	(no_connect
 		(at 63.5 179.07)
 	)
@@
 	(wire
 		(pts
+			(xy 93.98 158.75) (xy 105.41 158.75)
+		)
+		(stroke
+			(width 0)
+			(type default)
+		)
+	)
+	(wire
+		(pts
 			(xy 252.73 99.06) (xy 252.73 100.33)
 		)
@@
 	(hierarchical_label "~{5V_ON_OUT}"
 		(shape output)
-		(at 105.41 153.67 0)
+		(at 105.41 161.29 0)
 		(effects
 			(font
@@
 		)
 	)
+	(hierarchical_label "SOM_RST"
+		(shape output)
+		(at 105.41 158.75 0)
+		(effects
+			(font
+				(size 1.27 1.27)
+			)
+			(justify left)
+		)
+	)
 	(hierarchical_label "~{5V_ON_REQ}"
 		(shape input)
-		(at 105.41 161.29 0)
+		(at 105.41 153.67 0)
 		(effects
 			(font

Commit message: Fixed capacitors for the BQ25792
Parts:
- removed C17: 10u, Capacitor_SMD:C_0805_2012Metric, symbol Device:C
- removed C20: 100n, Capacitor_SMD:C_0402_1005Metric, symbol Device:C
