File: rf.kicad_sch (KiCad schematic)
At the start: 30 parts, among them IC1 SX1255IWLTRT, J1 Antenna, U2 BGS12P2L6, Y1 32MHz

Commit message: Added footprint of the SMA connector
The SMA connector is the original one used in Retevis C62. Dimensions
are based on measurements of the real part.
Parts:
- J1: footprint (none) -> parts:Connector_SMA_4x10mm
Changed lines of the file:
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@@
 			)
 		)
-		(property "Footprint" ""
+		(property "Footprint" "parts:Connector_SMA_4x10mm"
 			(at 252.73 83.82 0)
 			(effects

Commit message: Assigned missing footprints
Parts:
- L1, L2: footprint (none) -> Inductor_SMD:L_0603_1608Metric
Changed lines of the file:
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@@
 			)
 		)
-		(property "Footprint" ""
+		(property "Footprint" "Inductor_SMD:L_0603_1608Metric"
 			(at 144.78 45.72 0)
 			(effects
@@
 			)
 		)
-		(property "Footprint" ""
+		(property "Footprint" "Inductor_SMD:L_0603_1608Metric"
 			(at 139.7 50.8 0)
 			(effects

Commit message: Swapped RF inputs of the BGS12P2L6 for better PCB routing
Connections:
- net RF_IN: now also U2.1 (RF_OUT_2); no longer U2.3 (RF_OUT_1)
- net at C14.2: now also U2.3 (RF_OUT_1); no longer U2.1 (RF_OUT_2)
Other:
- moved on the sheet: C14
Changed lines of the file:
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@@
 	(wire
 		(pts
-			(xy 177.8 87.63) (xy 181.61 87.63)
+			(xy 177.8 80.01) (xy 181.61 80.01)
 		)
 		(stroke
@@
 	(wire
 		(pts
-			(xy 177.8 80.01) (xy 189.23 80.01)
+			(xy 177.8 87.63) (xy 189.23 87.63)
 		)
 		(stroke
@@
 	(wire
 		(pts
-			(xy 186.69 87.63) (xy 189.23 87.63)
+			(xy 186.69 80.01) (xy 189.23 80.01)
 		)
 		(stroke
@@
 	)
 	(label "RF_IN"
-		(at 177.8 80.01 180)
+		(at 177.8 87.63 180)
 		(effects
 			(font
@@
 	)
 	(label "RF_OUT"
-		(at 177.8 87.63 180)
+		(at 177.8 80.01 180)
 		(effects
 			(font
@@
 		(length 2.54)
 		(shape round)
-		(at 187.96 87.63 0)
+		(at 187.96 80.01 0)
 		(effects
 			(font
@@
 		)
 		(property "Netclass" "RF"
-			(at 186.69 83.312 0)
+			(at 186.69 75.692 0)
 			(effects
 				(font
@@
 		)
 		(property "Component Class" ""
-			(at 118.11 21.59 0)
+			(at 118.11 13.97 0)
 			(effects
 				(font
@@
 		(length 2.54)
 		(shape round)
-		(at 187.96 80.01 0)
+		(at 187.96 87.63 0)
 		(effects
 			(font
@@
 		)
 		(property "Netclass" "RF"
-			(at 186.69 75.692 0)
+			(at 186.69 83.312 0)
 			(effects
 				(font
@@
 		)
 		(property "Component Class" ""
-			(at 118.11 13.97 0)
+			(at 118.11 21.59 0)
 			(effects
 				(font
@@
 		(length 2.54)
 		(shape round)
-		(at 180.34 87.63 0)
+		(at 180.34 80.01 0)
 		(effects
 			(font
@@
 		)
 		(property "Netclass" "RF"
-			(at 179.07 83.312 0)
+			(at 179.07 75.692 0)
 			(effects
 				(font
@@
 		)
 		(property "Component Class" ""
-			(at 110.49 21.59 0)
+			(at 110.49 13.97 0)
 			(effects
 				(font
@@
 	(symbol
 		(lib_id "Device:C_Small")
-		(at 184.15 87.63 90)
+		(at 184.15 80.01 90)
 		(unit 1)
 		(exclude_from_sim no)
@@
 		(fields_autoplaced yes)
 		(property "Reference" "C14"
-			(at 184.1563 81.9234 90)
+			(at 184.1563 74.3034 90)
 			(effects
 				(font
@@
 		)
 		(property "Value" "1n"
-			(at 184.1563 84.3477 90)
+			(at 184.1563 76.7277 90)
 			(effects
 				(font
@@
 		)
 		(property "Footprint" "Capacitor_SMD:C_0402_1005Metric"
-			(at 184.15 87.63 0)
+			(at 184.15 80.01 0)
 			(effects
 				(font
@@
 		)
 		(property "Datasheet" "~"
-			(at 184.15 87.63 0)
+			(at 184.15 80.01 0)
 			(effects
 				(font
@@
 		)
 		(property "Description" ""
-			(at 184.15 87.63 0)
+			(at 184.15 80.01 0)
 			(effects
 				(font
@@
 		)
 		(property "PN" ""
-			(at 184.15 87.63 0)
+			(at 184.15 80.01 0)
 			(effects
 				(font
@@
 		)
 		(property "MPN" ""
-			(at 184.15 87.63 0)
+			(at 184.15 80.01 0)
 			(effects
 				(font
