File: soc.kicad_sch (KiCad schematic)
At the start: 5 parts, among them U1 MCM-iMX93

Commit message: Added BOM assigment for most of the parts
Parts:
- R1: LCSC (none) -> C25752; PN (none) -> 0402WGF1202TCE
- R2: LCSC (none) -> C25768; PN (none) -> 0402WGF2202TCE
- R3, R4: LCSC (none) -> C25152; PN (none) -> 0402WGJ0220TCE
- U1: now left out of the parts list
Changed lines of the file:
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@@
 			)
 		)
-		(property "PN" ""
+		(property "PN" "0402WGJ0220TCE"
 			(at 50.8 36.83 0)
 			(effects
@@
 		(property "MPN" ""
 			(at 50.8 36.83 0)
+			(effects
+				(font
+					(size 1.27 1.27)
+				)
+				(hide yes)
+			)
+		)
+		(property "LCSC" "C25152"
+			(at 50.8 36.83 90)
 			(effects
 				(font
@@
 		(unit 1)
 		(exclude_from_sim no)
-		(in_bom yes)
+		(in_bom no)
 		(on_board yes)
 		(dnp no)
@@
 			)
 		)
-		(property "PN" ""
+		(property "PN" "0402WGF2202TCE"
 			(at 38.1 44.45 0)
 			(effects
@@
 		(property "MPN" ""
 			(at 38.1 44.45 0)
+			(effects
+				(font
+					(size 1.27 1.27)
+				)
+				(hide yes)
+			)
+		)
+		(property "LCSC" "C25768"
+			(at 38.1 44.45 90)
 			(effects
 				(font
@@
 			)
 		)
-		(property "PN" ""
+		(property "PN" "0402WGF1202TCE"
 			(at 38.1 36.83 0)
 			(effects
@@
 		(property "MPN" ""
 			(at 38.1 36.83 0)
+			(effects
+				(font
+					(size 1.27 1.27)
+				)
+				(hide yes)
+			)
+		)
+		(property "LCSC" "C25752"
+			(at 38.1 36.83 90)
 			(effects
 				(font
@@
 			)
 		)
-		(property "PN" ""
+		(property "PN" "0402WGJ0220TCE"
 			(at 53.34 36.83 0)
 			(effects
@@
 			(effects
 				(font
+					(size 1.27 1.27)
+				)
+				(hide yes)
+			)
+		)
+		(property "LCSC" "C25152"
+			(at 53.34 36.83 90)
+			(effects
+				(font

Commit message: Added 4 decoupling capacitors to the SoM `V_SOM` pins
Fixes #30
Parts:
- removed R3, R4: 22R, Resistor_SMD:R_0402_1005Metric, symbol Device:R_Small
- added C62, C63, C64, C65: 100n, Capacitor_SMD:C_0402_1005Metric, symbol Device:C
Connections:
- net +5V: now also C62.1, C63.1, C64.1, C65.1
- net GND: now also C62.2, C63.2, C64.2, C65.2
- net USB_DN: now also U1.140 (USB1_DN)
- net USB_DP: now also U1.139 (USB1_DP)
Other:
- note added: "Decoupling capacitors, as close to the V_SOM pins as possible."

Commit message: Replaced WM8960 to the newer TLV320AIC3100
WM8960 is obsolete, so this change is needed.
Fixes #29
Connections:
- net MIC_GAIN renamed JACK_DETECT
- net ~{MIC_MUTE}: no longer names the net of U1.68 (GPIO3_IO[5])
- no-connect marks 82 -> 83
Changed lines of the file:
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@@
 	)
 	(no_connect
+		(at 132.08 171.45)
+	)
+	(no_connect
 		(at 60.96 45.72)
 	)
@@
 	(wire
 		(pts
-			(xy 132.08 171.45) (xy 132.08 177.8)
-		)
-		(stroke
-			(width 0)
-			(type default)
-		)
-	)
-	(wire
-		(pts
 			(xy 86.36 40.64) (xy 86.36 45.72)
 		)
@@
 		)
 	)
-	(hierarchical_label "~{MIC_MUTE}"
-		(shape output)
-		(at 132.08 177.8 270)
-		(effects
-			(font
-				(size 1.27 1.27)
-			)
-			(justify right)
-		)
-	)
 	(hierarchical_label "SPI0_MISO"
 		(shape input)
@@
 		)
 	)
-	(hierarchical_label "MIC_GAIN"
-		(shape output)
-		(at 129.54 177.8 270)
-		(effects
-			(font
-				(size 1.27 1.27)
-			)
-			(justify right)
-		)
-	)
 	(hierarchical_label "~{RST}"
 		(shape input)
@@
 		)
 	)
+	(hierarchical_label "JACK_DETECT"
+		(shape input)
+		(at 129.54 177.8 270)
+		(effects
+			(font
+				(size 1.27 1.27)
+			)
+			(justify right)
+		)
+	)
 	(hierarchical_label "RF_RST"
 		(shape output)
@@
 			)
 		)
+		(property "LCSC Part" ""
+			(at 234.95 64.77 0)
+			(effects
+				(font
+					(size 1.27 1.27)
+				)
+				(hide yes)
+			)
+		)
 		(pin "1"
 		)
@@
 			)
 		)
+		(property "LCSC Part" ""
+			(at 196.85 64.77 0)
+			(effects
+				(font
+					(size 1.27 1.27)
+				)
+				(hide yes)
+			)
+		)
 		(pin "1"
 		)
@@
 			)
 		)
+		(property "LCSC Part" ""
+			(at 93.98 105.41 0)
+			(effects
+				(font
+					(size 1.27 1.27)
+				)
+				(hide yes)
+			)
+		)
 		(pin "6"
 		)
@@
 			)
 		)
+		(property "LCSC Part" ""
+			(at 38.1 44.45 90)
+			(effects
+				(font
+					(size 1.27 1.27)
+				)
+				(hide yes)
+			)
+		)
 		(pin "1"
 		)
@@
 			)
 		)
+		(property "LCSC Part" ""
+			(at 222.25 64.77 0)
+			(effects
+				(font
+					(size 1.27 1.27)
+				)
+				(hide yes)
+			)
+		)
 		(pin "1"
 		)
@@
 			)
 		)
+		(property "LCSC Part" ""
+			(at 38.1 36.83 90)
+			(effects
+				(font
+					(size 1.27 1.27)
+				)
+				(hide yes)
+			)
+		)
 		(pin "1"
 		)
@@
 			(at 209.55 64.77 0)
 			(effects
+				(font
+					(size 1.27 1.27)
+				)
+				(hide yes)
+			)
+		)
+		(property "LCSC Part" ""
+			(at 209.55 64.77 0)
+			(effects
