File: soc.kicad_sch (KiCad schematic)
At the start: 7 parts, among them U1 MCM-iMX93

Commit message: Fixed and added LCSC reference numbers for all components
Parts:
- R1: MPN (none) -> 0402WGF1202TCE; PN 0402WGF1202TCE -> (none)
- R2: MPN (none) -> 0402WGF2202TCE; PN 0402WGF2202TCE -> (none)
Changed lines of the file:
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@@
 			)
 		)
-		(property "PN" "0402WGF2202TCE"
+		(property "PN" ""
 			(at 38.1 44.45 0)
 			(effects
@@
 			)
 		)
-		(property "MPN" ""
+		(property "MPN" "0402WGF2202TCE"
 			(at 38.1 44.45 0)
 			(effects
@@
 			)
 		)
-		(property "PN" "0402WGF1202TCE"
+		(property "PN" ""
 			(at 38.1 36.83 0)
 			(effects
@@
 			)
 		)
-		(property "MPN" ""
+		(property "MPN" "0402WGF1202TCE"
 			(at 38.1 36.83 0)
 			(effects

Commit message: Removed unused components, connected power signals to the SoM
Connections:
- net 3V3_ON_REQ: now reaches U1.103 (GPIO2_IO[15])
- no-connect marks 83 -> 82
Changed lines of the file:
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@@
-	)
-	(no_connect
-		(at 143.51 67.31)
 	)
 	(no_connect
@@
 		(pts
 			(xy 234.95 68.58) (xy 234.95 69.85)
+		)
+		(stroke
+			(width 0)
+			(type default)
+		)
+	)
+	(wire
+		(pts
+			(xy 143.51 67.31) (xy 148.59 67.31)
 		)
 		(stroke
@@
 		(effects
 			(font
+				(size 1.27 1.27)
+			)
+			(justify left)
+		)
+	)
+	(hierarchical_label "3V3_ON_REQ"
+		(shape output)
+		(at 148.59 67.31 0)
+		(effects
+			(font

Commit message: Added power management ATTiny826
Fixes #32
Fixes #35
Fixes #23
Parts:
- added C25: 100n, Capacitor_SMD:C_0402_1005Metric, symbol Device:C
Connections:
- net 3V3_ON_REQ is gone; now on net ON/OFF: U1.103 (GPIO2_IO[15])
- net ON/OFF_SW is gone; now on net +5V: U1.102 (GPIO2_IO[14])
- net VOL_BATT is gone; now on net I2C_SCL: U1.9
- net +5V: now also U1.100 (SAI3_MCLK), U1.91, U1.95; no longer U1.11 (V_SOM), U1.15 (V_SOM), U1.4 (V_SOM), U1.6 (V_SOM)
- net D1: now also U1.55 (GPIO4_IO[17]); no longer U1.51 (GPIO4_IO[16])
- net D2: now also U1.54 (GPIO4_IO[20]); no longer U1.52 (GPIO4_IO[19])
- net D4: now also U1.52 (GPIO4_IO[19]); no longer U1.54 (GPIO4_IO[20])
- net D5: now also U1.51 (GPIO4_IO[16]); no longer U1.55 (GPIO4_IO[17])
- net D6: now also U1.50; no longer U1.56 (GPIO4_IO[21])
- net D7: now also U1.49; no longer U1.57 (GPIO4_IO[23])
- net D8: now also U1.48; no longer U1.58 (GPIO4_IO[22])
- net D9: now also U1.47 (SAI3_TX_SYNC); no longer U1.59 (GPIO4_IO[24])
- net EXT_PTT: now also U1.134 (VSD_3V3); no longer U1.112 (GPIO3_IO[23)
- net GND: now also U1.31, C25.2
- net I2C_SCL: no longer U1.97 (GPIO2_IO[29])
- net I2C_SDA: now also U1.8; no longer U1.98 (GPIO2_IO[28])
- net I2S0_CLK: now also U1.114 (GPIO3_IO[22]); no longer U1.132 (SAI1_TX_BCLK)
- net I2S0_DIN: now also U1.115 (GPIO2_IO[22]); no longer U1.131 (SAI1_RX_DATA[0])
- net I2S0_DOUT: now also U1.40; no longer U1.66 (SAI1_TX_DATA[0])
- net I2S0_WS: now also U1.120 (GPIO2_IO[8]); no longer U1.126 (SAI1_TX_SYNC)
- net I2S1_CLK: now also U1.5 (ALT_BOOT_USB); no longer U1.101 (SAI3_TX_BCLK)
- net I2S1_DIN: now also U1.130; no longer U1.116 (SAI3_RX_DATA[0])
- net I2S1_DOUT: now also U1.129 (GPIO2_IO[0]); no longer U1.117 (SAI3_TX_DATA[0])
- net I2S1_MCLK: now also U1.6 (V_SOM); no longer U1.100 (SAI3_MCLK)
- net I2S1_WS: now also U1.59 (GPIO4_IO[24]); no longer U1.47 (SAI3_TX_SYNC)
- net INT_PTT: now also U1.133; no longer U1.113 (GPIO3_IO[21])
- net JACK_DETECT: now also U1.39; no longer U1.67 (GPIO3_IO[6])
- net KBD_PWM: now also U1.1 (USB1_ID); no longer U1.105 (GPIO2_IO[12])
- net LCD_PWM: now also U1.7; no longer U1.99 (GPIO2_IO[24])
- net LCD_RS: now also U1.127 (VCC_RTC); no longer U1.119 (GPIO2_IO[19])
- net LED_A: now also U1.122 (SPI3_SCK); no longer U1.124 (GPIO2_IO[5])
- net LED_B: now also U1.121 (SPI3_SIN); no longer U1.125 (GPIO2_IO[4])
- net LIGHT: now also U1.128 (SPI6_SOUT); no longer U1.118 (GPIO2_IO[18])
- net ON/OFF: no longer U1.3 (ON/OFF)
- net RF_RST: now also U1.131 (SAI1_RX_DATA[0]); no longer U1.115 (GPIO2_IO[22])
- net RF_SW_CTRL: now also U1.2 (USB1_VBUS_3V3); no longer U1.104 (GPIO2_IO[13])
- net SIDE_BTN: now also U1.132 (SAI1_TX_BCLK); no longer U1.114 (GPIO3_IO[22])
- net SPI0_MISO: now also U1.125 (GPIO2_IO[4]); no longer U1.121 (SPI3_SIN)
- net SPI0_SCK: now also U1.124 (GPIO2_IO[5]); no longer U1.122 (SPI3_SCK)
- net SPI1_MISO: now also U1.61 (GPIO4_IO[26]); no longer U1.45 (SPI6_SIN)
- net SPI1_MOSI: now also U1.118 (GPIO2_IO[18]); no longer U1.128 (SPI6_SOUT)
- net SPI1_SCK: now also U1.138; no longer U1.108 (SPI6_SCK)
- net SPI_CS_LCD: now also U1.117 (SAI3_TX_DATA[0]); no longer U1.129 (GPIO2_IO[0])
- net SPI_CS_RF: now also U1.126 (SAI1_TX_SYNC); no longer U1.120 (GPIO2_IO[8])
- net STBY: now also U1.90; no longer U1.16 (PMIC_STBY_REQ)
- net UART_RX: now also U1.42; no longer U1.64 (UART1_RX)
- net UART_TX: now also U1.43; no longer U1.63 (UART1_TX)
- net USB_BOOT: now also U1.101 (SAI3_TX_BCLK); no longer U1.5 (ALT_BOOT_USB)
- net USB_DN: now also U1.106; no longer U1.140 (USB1_DN)
- net USB_DP: now also U1.107; no longer U1.139 (USB1_DP)
- net VOL_POT: now also U1.96; no longer U1.10 (VOL_ADC)
- net ~{RST}: now also U1.92; no longer U1.14 (SYS_NRST)
- net at R1.1, R2.2: now also U1.104 (GPIO2_IO[13]); no longer U1.2 (USB1_VBUS_3V3)
- new net +3.3VP: C25.1, U1.119 (GPIO2_IO[19])
- no-connect marks 82 -> 84

Commit message: Changed 5V DC/DC buck to TPS565242
Original buck has 2 A maximum current output. New one has up to 5 A.
Our design needs ~3 A maximum current.

Fixes #38
Connections:
- net +3.3VP: now also U1.127 (VCC_RTC); no longer U1.119 (GPIO2_IO[19])
- net +5V: now also U1.11 (V_SOM), U1.15 (V_SOM), U1.4 (V_SOM), U1.6 (V_SOM); no longer U1.100 (SAI3_MCLK), U1.102 (GPIO2_IO[14]), U1.91, U1.95
- net D1: now also U1.51 (GPIO4_IO[16]); no longer U1.55 (GPIO4_IO[17])
- net D2: now also U1.52 (GPIO4_IO[19]); no longer U1.54 (GPIO4_IO[20])
- net D4: now also U1.54 (GPIO4_IO[20]); no longer U1.52 (GPIO4_IO[19])
- net D5: now also U1.55 (GPIO4_IO[17]); no longer U1.51 (GPIO4_IO[16])
- net D6: now also U1.56 (GPIO4_IO[21]); no longer U1.50
- net D7: now also U1.57 (GPIO4_IO[23]); no longer U1.49
- net D8: now also U1.58 (GPIO4_IO[22]); no longer U1.48
- net D9: now also U1.59 (GPIO4_IO[24]); no longer U1.47 (SAI3_TX_SYNC)
- net EXT_PTT: now also U1.112 (GPIO3_IO[23); no longer U1.134 (VSD_3V3)
- net GND: no longer U1.31
- net I2C_SCL: now also U1.97 (GPIO2_IO[29]); no longer U1.9
- net I2C_SDA: now also U1.98 (GPIO2_IO[28]); no longer U1.8
- net I2S0_CLK: now also U1.132 (SAI1_TX_BCLK); no longer U1.114 (GPIO3_IO[22])
- net I2S0_DIN: now also U1.131 (SAI1_RX_DATA[0]); no longer U1.115 (GPIO2_IO[22])
- net I2S0_DOUT: now also U1.66 (SAI1_TX_DATA[0]); no longer U1.40
- net I2S0_WS: now also U1.126 (SAI1_TX_SYNC); no longer U1.120 (GPIO2_IO[8])
- net I2S1_CLK: now also U1.101 (SAI3_TX_BCLK); no longer U1.5 (ALT_BOOT_USB)
- net I2S1_DIN: now also U1.116 (SAI3_RX_DATA[0]); no longer U1.130
- net I2S1_DOUT: now also U1.117 (SAI3_TX_DATA[0]); no longer U1.129 (GPIO2_IO[0])
- net I2S1_MCLK: now also U1.100 (SAI3_MCLK); no longer U1.6 (V_SOM)
- net I2S1_WS: now also U1.47 (SAI3_TX_SYNC); no longer U1.59 (GPIO4_IO[24])
- net INT_PTT: now also U1.113 (GPIO3_IO[21]); no longer U1.133
- net JACK_DETECT: now also U1.67 (GPIO3_IO[6]); no longer U1.39
- net KBD_PWM: now also U1.105 (GPIO2_IO[12]); no longer U1.1 (USB1_ID)
- net LCD_PWM: now also U1.99 (GPIO2_IO[24]); no longer U1.7
- net LCD_RS: now also U1.119 (GPIO2_IO[19]); no longer U1.127 (VCC_RTC)
- net LED_A: now also U1.124 (GPIO2_IO[5]); no longer U1.122 (SPI3_SCK)
- net LED_B: now also U1.125 (GPIO2_IO[4]); no longer U1.121 (SPI3_SIN)
- net LIGHT: now also U1.118 (GPIO2_IO[18]); no longer U1.128 (SPI6_SOUT)
- net ON/OFF: now also U1.3 (ON/OFF); no longer U1.103 (GPIO2_IO[15])
- net RF_RST: now also U1.115 (GPIO2_IO[22]); no longer U1.131 (SAI1_RX_DATA[0])
- net RF_SW_CTRL: now also U1.104 (GPIO2_IO[13]); no longer U1.2 (USB1_VBUS_3V3)
- net SIDE_BTN: now also U1.114 (GPIO3_IO[22]); no longer U1.132 (SAI1_TX_BCLK)
- net SPI0_MISO: now also U1.121 (SPI3_SIN); no longer U1.125 (GPIO2_IO[4])
- net SPI0_SCK: now also U1.122 (SPI3_SCK); no longer U1.124 (GPIO2_IO[5])
- net SPI1_MISO: now also U1.45 (SPI6_SIN); no longer U1.61 (GPIO4_IO[26])
- net SPI1_MOSI: now also U1.128 (SPI6_SOUT); no longer U1.118 (GPIO2_IO[18])
- net SPI1_SCK: now also U1.108 (SPI6_SCK); no longer U1.138
- net SPI_CS_LCD: now also U1.129 (GPIO2_IO[0]); no longer U1.117 (SAI3_TX_DATA[0])
- net SPI_CS_RF: now also U1.120 (GPIO2_IO[8]); no longer U1.126 (SAI1_TX_SYNC)
- net STBY: now also U1.16 (PMIC_STBY_REQ); no longer U1.90
- net UART_RX: now also U1.64 (UART1_RX); no longer U1.42
- net UART_TX: now also U1.63 (UART1_TX); no longer U1.43
- net USB_BOOT: now also U1.5 (ALT_BOOT_USB); no longer U1.101 (SAI3_TX_BCLK)
- net USB_DN: now also U1.140 (USB1_DN); no longer U1.106
- net USB_DP: now also U1.139 (USB1_DP); no longer U1.107
- net VOL_POT: now also U1.10 (VOL_ADC); no longer U1.96
- net ~{RST}: now also U1.14 (SYS_NRST); no longer U1.92
- net at R1.1, R2.2: now also U1.2 (USB1_VBUS_3V3); no longer U1.104 (GPIO2_IO[13])
Changed lines of the file:
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@@
 		(lib_id "MCM-iMX93-SOM:MCM-iMX93-SOM")
 		(at 93.98 105.41 0)
-		(mirror y)
 		(unit 1)
 		(exclude_from_sim no)

Commit message: Added test point for the USB ID SoM pin
Parts:
- added TP12: USB_ID, TestPoint:TestPoint_Pad_D1.0mm, symbol Connector:TestPoint_Alt
Connections:
- net at U1.1 (USB1_ID): now also TP12.1
- no-connect marks 84 -> 83
Other:
- moved on the sheet: R1, R2
Changed lines of the file:
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@@
 	(text "USB_ID NC"
 		(exclude_from_sim no)
-		(at 31.75 62.23 0)
+		(at 27.94 62.484 0)
 		(effects
 			(font
@@
 	)
 	(junction
-		(at 38.1 40.64)
+		(at 30.48 40.64)
 		(diameter 0)
 		(color 0 0 0 0)
@@
 	)
 	(no_connect
-		(at 44.45 62.23)
-	)
-	(no_connect
 		(at 58.42 171.45)
 	)
@@
 	(wire
 		(pts
-			(xy 38.1 46.99) (xy 38.1 48.26)
+			(xy 30.48 46.99) (xy 30.48 48.26)
 		)
 		(stroke
@@
 	(wire
 		(pts
-			(xy 41.91 64.77) (xy 41.91 40.64)
+			(xy 34.29 64.77) (xy 34.29 40.64)
 		)
 		(stroke
@@
 	(wire
 		(pts
-			(xy 38.1 39.37) (xy 38.1 40.64)
+			(xy 30.48 39.37) (xy 30.48 40.64)
 		)
 		(stroke
@@
 	(wire
 		(pts
+			(xy 41.91 62.23) (xy 44.45 62.23)
+		)
+		(stroke
+			(width 0)
+			(type default)
+		)
+	)
+	(wire
+		(pts
 			(xy 109.22 40.64) (xy 109.22 45.72)
 		)
@@
 	(wire
 		(pts
-			(xy 34.29 33.02) (xy 38.1 33.02)
+			(xy 26.67 33.02) (xy 30.48 33.02)
 		)
 		(stroke
@@
 	(wire
 		(pts
-			(xy 38.1 40.64) (xy 38.1 41.91)
+			(xy 30.48 40.64) (xy 30.48 41.91)
 		)
 		(stroke
@@
 	(wire
 		(pts
-			(xy 38.1 33.02) (xy 38.1 34.29)
+			(xy 30.48 33.02) (xy 30.48 34.29)
 		)
 		(stroke
@@
 	(wire
 		(pts
-			(xy 44.45 64.77) (xy 41.91 64.77)
+			(xy 44.45 64.77) (xy 34.29 64.77)
 		)
 		(stroke
@@
 	(wire
 		(pts
-			(xy 41.91 40.64) (xy 38.1 40.64)
+			(xy 34.29 40.64) (xy 30.48 40.64)
 		)
 		(stroke
@@
 	(hierarchical_label "USB_VSENSE"
 		(shape input)
-		(at 34.29 33.02 180)
+		(at 26.67 33.02 180)
 		(effects
 			(font
@@
 	)
 	(symbol
+		(lib_id "Connector:TestPoint_Alt")
+		(at 41.91 62.23 90)
+		(mirror x)
+		(unit 1)
+		(exclude_from_sim no)
+		(in_bom no)
+		(on_board yes)
+		(dnp no)
+		(property "Reference" "TP12"
+			(at 41.656 57.912 90)
+			(effects
+				(font
+					(size 1.27 1.27)
+				)
+				(justify left)
+			)
+		)
+		(property "Value" "USB_ID"
+			(at 42.418 59.944 90)
+			(effects
+				(font
+					(size 1.27 1.27)
+				)
+				(justify left)
+			)
+		)
+		(property "Footprint" "TestPoint:TestPoint_Pad_D1.0mm"
+			(at 41.91 67.31 0)
+			(effects
+				(font
+					(size 1.27 1.27)
+				)
+				(hide yes)
+			)
+		)
+		(property "Datasheet" "~"
+			(at 41.91 67.31 0)
+			(effects
+				(font
+					(size 1.27 1.27)
+				)
+				(hide yes)
+			)
+		)
+		(property "Description" "test point (alternative shape)"
+			(at 41.91 62.23 0)
+			(effects
+				(font
+					(size 1.27 1.27)
+				)
+				(hide yes)
+			)
+		)
+		(property "LCSC Part" ""
+			(at 41.91 62.23 90)
+			(effects
+				(font
+					(size 1.27 1.27)
+				)
+				(hide yes)
+			)
+		)
+		(pin "1"
+		)
+		(instances
+			(project "linht-hw"
+				(path "/73efc1fc-21f6-4aef-9f73-508fe18fa32e/9e50fe40-00b4-48a0-8ec6-ce79209e6a2d"
+					(reference "TP12")
+					(unit 1)
+				)
+			)
+		)
+	)
+	(symbol
 		(lib_id "power:+5V")
 		(at 36.83 78.74 0)
@@
 	(symbol
 		(lib_id "Device:R_Small")
-		(at 38.1 44.45 180)
+		(at 30.48 44.45 180)
 		(unit 1)
 		(exclude_from_sim no)
@@
 		(dnp no)
 		(property "Reference" "R2"
-			(at 35.56 44.45 90)
+			(at 27.94 44.45 90)
 			(effects
 				(font
@@
 		)
 		(property "Value" "22k"
-			(at 40.64 44.45 90)
+			(at 33.02 44.45 90)
 			(effects
 				(font
@@
 		)
 		(property "Footprint" "Resistor_SMD:R_0402_1005Metric"
-			(at 38.1 44.45 0)
+			(at 30.48 44.45 0)
 			(effects
 				(font
@@
 		)
 		(property "Datasheet" "~"
-			(at 38.1 44.45 0)
+			(at 30.48 44.45 0)
 			(effects
 				(font
@@
 		)
 		(property "Description" "Resistor, small symbol"
-			(at 38.1 44.45 0)
+			(at 30.48 44.45 0)
 			(effects
 				(font
@@
 		)
 		(property "PN" ""
-			(at 38.1 44.45 0)
+			(at 30.48 44.45 0)
 			(effects
 				(font
@@
 		)
 		(property "MPN" "0402WGF2202TCE"
-			(at 38.1 44.45 0)
+			(at 30.48 44.45 0)
 			(effects
 				(font
@@
 		)
 		(property "LCSC" "C25768"
-			(at 38.1 44.45 90)
+			(at 30.48 44.45 90)
 			(effects
 				(font
@@
 		)
 		(property "LCSC Part" ""
-			(at 38.1 44.45 90)
+			(at 30.48 44.45 90)
 			(effects
 				(font
@@
 	(symbol
 		(lib_id "power:GND")
-		(at 38.1 48.26 0)
+		(at 30.48 48.26 0)
 		(unit 1)
 		(exclude_from_sim no)
@@
 		(fields_autoplaced yes)
 		(property "Reference" "#PWR02"
-			(at 38.1 54.61 0)
+			(at 30.48 54.61 0)
 			(effects
 				(font
@@
 		)
 		(property "Value" "GND"
-			(at 38.1 52.3931 0)
+			(at 30.48 52.3931 0)
 			(effects
 				(font
@@
 		)
 		(property "Footprint" ""
-			(at 38.1 48.26 0)
+			(at 30.48 48.26 0)
 			(effects
 				(font
@@
 		)
 		(property "Datasheet" ""
-			(at 38.1 48.26 0)
+			(at 30.48 48.26 0)
 			(effects
 				(font
@@
 		)
 		(property "Description" "Power symbol creates a global label with name \"GND\" , ground"
-			(at 38.1 48.26 0)
+			(at 30.48 48.26 0)
 			(effects
 				(font
@@
 	(symbol
 		(lib_id "Device:R_Small")
-		(at 38.1 36.83 180)
+		(at 30.48 36.83 180)
 		(unit 1)
 		(exclude_from_sim no)
@@
 		(dnp no)
 		(property "Reference" "R1"
-			(at 35.56 36.83 90)
+			(at 27.94 36.83 90)
 			(effects
 				(font
@@
 		)
 		(property "Value" "12k"
-			(at 40.64 36.83 90)
+			(at 33.02 36.83 90)
 			(effects
 				(font
@@
 		)
 		(property "Footprint" "Resistor_SMD:R_0402_1005Metric"
-			(at 38.1 36.83 0)
+			(at 30.48 36.83 0)
 			(effects
 				(font
@@
 		)
 		(property "Datasheet" "~"
-			(at 38.1 36.83 0)
+			(at 30.48 36.83 0)
 			(effects
 				(font
@@
 		)
 		(property "Description" "Resistor, small symbol"
-			(at 38.1 36.83 0)
+			(at 30.48 36.83 0)
 			(effects
 				(font
@@
 		)
 		(property "PN" ""
-			(at 38.1 36.83 0)
+			(at 30.48 36.83 0)
 			(effects
 				(font
@@
 		)
 		(property "MPN" "0402WGF1202TCE"
-			(at 38.1 36.83 0)
+			(at 30.48 36.83 0)
 			(effects
 				(font
@@
 		)
 		(property "LCSC" "C25752"
-			(at 38.1 36.83 90)
+			(at 30.48 36.83 90)
 			(effects
 				(font
@@
 		)
 		(property "LCSC Part" ""
-			(at 38.1 36.83 90)
+			(at 30.48 36.83 90)
 			(effects
 				(font

Commit message: Changed GPIO for the jack detect signal to pin 49
Connections:
- net JACK_DETECT: now also U1.49; no longer U1.67 (GPIO3_IO[6])
Changed lines of the file:
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@@
-	)
-	(no_connect
-		(at 83.82 171.45)
 	)
 	(no_connect
@@
 	(no_connect
 		(at 143.51 148.59)
+	)
+	(no_connect
+		(at 129.54 171.45)
 	)
 	(no_connect
@@
 	(wire
 		(pts
-			(xy 129.54 171.45) (xy 129.54 177.8)
+			(xy 83.82 171.45) (xy 83.82 177.8)
 		)
 		(stroke
@@
 	(hierarchical_label "JACK_DETECT"
 		(shape input)
-		(at 129.54 177.8 270)
-		(effects
-			(font
+		(at 83.82 177.8 270)
+		(effects
+			(font

Commit message: Connected attenuator data signals to SoM and minor changes to SoM pinout
KBD_PWM from 105  -> 95  (GPIO2_IO[25])
RF_SW_CTRL from 104 -> 103 (GPIO2_IO[15])
RF_ATT_DATA to 107 (SPI7_SOUT)
RF_ATT_CLK to 106 (SPI7_SCK)
RF_ATT_LE1 to 105 (GPIO2_IO[12])
RF_ATT_LE2 to 104 (GPIO2_IO[13])
RF_PA_SHUTDOWN not decided yet
Connections:
- net KBD_PWM: now also U1.95; no longer U1.105 (GPIO2_IO[12])
- net RF_SW_CTRL: now also U1.103 (GPIO2_IO[15]); no longer U1.104 (GPIO2_IO[13])
- net RF_ATT_CLK: now reaches U1.106
- net RF_ATT_DATA: now reaches U1.107
- new net RF_ATT_LE1: U1.105 (GPIO2_IO[12])
- new net RF_ATT_LE2: U1.104 (GPIO2_IO[13])
- no-connect marks 83 -> 79
Changed lines of the file:
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@@
-	)
-	(no_connect
-		(at 143.51 87.63)
 	)
 	(no_connect
@@
 	)
 	(no_connect
-		(at 134.62 45.72)
-	)
-	(no_connect
 		(at 63.5 45.72)
 	)
@@
 	)
 	(no_connect
-		(at 137.16 45.72)
-	)
-	(no_connect
 		(at 143.51 92.71)
 	)
@@
 	(no_connect
 		(at 44.45 133.35)
-	)
-	(no_connect
-		(at 143.51 67.31)
 	)
 	(no_connect
@@
 	(wire
 		(pts
+			(xy 143.51 62.23) (xy 148.59 62.23)
+		)
+		(stroke
+			(width 0)
+			(type default)
+		)
+	)
+	(wire
+		(pts
 			(xy 222.25 68.58) (xy 222.25 69.85)
 		)
@@
 	(wire
 		(pts
+			(xy 143.51 64.77) (xy 148.59 64.77)
+		)
+		(stroke
+			(width 0)
+			(type default)
+		)
+	)
+	(wire
+		(pts
 			(xy 41.91 74.93) (xy 44.45 74.93)
 		)
@@
 	(wire
 		(pts
+			(xy 134.62 40.64) (xy 134.62 45.72)
+		)
+		(stroke
+			(width 0)
+			(type default)
+		)
+	)
+	(wire
+		(pts
 			(xy 26.67 33.02) (xy 30.48 33.02)
 		)
@@
 	(wire
 		(pts
-			(xy 143.51 64.77) (xy 148.59 64.77)
+			(xy 143.51 67.31) (xy 148.59 67.31)
 		)
 		(stroke
@@
 	(wire
 		(pts
+			(xy 137.16 40.64) (xy 137.16 45.72)
+		)
+		(stroke
+			(width 0)
+			(type default)
+		)
+	)
+	(wire
+		(pts
 			(xy 93.98 171.45) (xy 93.98 175.26)
 		)
@@
 	(wire
 		(pts
-			(xy 143.51 62.23) (xy 148.59 62.23)
+			(xy 143.51 87.63) (xy 148.59 87.63)
 		)
 		(stroke
@@
 	(hierarchical_label "RF_SW_CTRL"
 		(shape output)
-		(at 148.59 64.77 0)
+		(at 148.59 67.31 0)
 		(effects
 			(font
@@
 	(hierarchical_label "KBD_PWM"
 		(shape output)
-		(at 148.59 62.23 0)
+		(at 148.59 87.63 0)
+		(effects
+			(font
+				(size 1.27 1.27)
+			)
+			(justify left)
+		)
+	)
+	(hierarchical_label "RF_ATT_LE2"
+		(shape input)
+		(at 148.59 64.77 0)
 		(effects
 			(font
@@
 		)
 	)
+	(hierarchical_label "RF_ATT_CLK"
+		(shape input)
+		(at 137.16 40.64 90)
+		(effects
+			(font
+				(size 1.27 1.27)
+			)
+			(justify left)
+		)
+	)
 	(hierarchical_label "SPI0_MOSI"
 		(shape output)
@@
 		)
 	)
+	(hierarchical_label "RF_ATT_DATA"
+		(shape input)
+		(at 134.62 40.64 90)
+		(effects
+			(font
+				(size 1.27 1.27)
+			)
+			(justify left)
+		)
+	)
 	(hierarchical_label "I2S1_WS"
 		(shape output)
@@
 		(effects
 			(font
+				(size 1.27 1.27)
+			)
+			(justify left)
+		)
+	)
+	(hierarchical_label "RF_ATT_LE1"
+		(shape input)
+		(at 148.59 62.23 0)
+		(effects
+			(font
