File: soc.kicad_sch (KiCad schematic)
At the start: 9 parts, among them U1 MCM-iMX93

Commit message: Add SoM MCM-iMC93 into the BOM
Parts:
- U1: MPN (none) -> MCM-iMX93-C1700D-D2-N32; now in the parts list
Changed lines of the file:
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@@
 		(unit 1)
 		(exclude_from_sim no)
-		(in_bom no)
+		(in_bom yes)
 		(on_board yes)
 		(dnp no)
@@
 			(at 93.98 105.41 0)
 			(effects
+				(font
+					(size 1.27 1.27)
+				)
+				(hide yes)
+			)
+		)
+		(property "MPN" "MCM-iMX93-C1700D-D2-N32"
+			(at 93.98 105.41 0)
+			(effects

Commit message: Add SoM part number to the PN field
Parts:
- U1: PN (none) -> MCM-iMX93-C1700D-D2-N32
Changed lines of the file:
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@@
+			)
+		)
+		(property "PN" "MCM-iMX93-C1700D-D2-N32"
+			(at 93.98 105.41 0)
+			(effects
+				(font
+					(size 1.27 1.27)
+				)
+				(hide yes)
 			)
 		)

Commit message: Fixed GNSS TX/RX mixup and several ERC issues
Connections:
- net GNSS_RX: now also U1.88; no longer U1.84
- net GNSS_TX: now also U1.84; no longer U1.88
Changed lines of the file:
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@@
 	(hierarchical_label "GNSS_TX"
 		(shape output)
-		(at 148.59 105.41 0)
+		(at 148.59 115.57 0)
 		(effects
 			(font
@@
 	(hierarchical_label "GNSS_RX"
 		(shape input)
-		(at 148.59 115.57 0)
+		(at 148.59 105.41 0)
 		(effects
 			(font
