File: gnss.kicad_sch (KiCad schematic)
At the start: 15 parts, among them U13 LG77L

Commit message: Fixed LG77L Mouser and LCSC part numbers
Parts:
- U13: MPN (none) -> LG77LICMD; PN (none) -> 277-LG77LICMD
Changed lines of the file:
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@@
+			)
+		)
+		(property "MPN" "LG77LICMD "
+			(at 140.97 115.57 0)
+			(effects
+				(font
+					(size 1.27 1.27)
+				)
+				(hide yes)
+			)
+		)
+		(property "PN" " 277-LG77LICMD"
+			(at 140.97 115.57 0)
+			(effects
+				(font
+					(size 1.27 1.27)
+				)
+				(hide yes)
 			)
 		)

Commit message: Remove whitespaces in PN and MPN fields
Parts:
- AE1: PN 603-ANT8010LL05R1516 -> 603-ANT8010LL05R1516
- C23, C93, C95: PN 187-CL05B104KO5NNNC -> 187-CL05B104KO5NNNC
- U13: PN 277-LG77LICMD -> 277-LG77LICMD
Changed lines of the file:
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@@
 			)
 		)
-		(property "PN" " 277-LG77LICMD"
+		(property "PN" "277-LG77LICMD"
 			(at 140.97 115.57 0)
 			(effects
@@
 			)
 		)
-		(property "PN" " 187-CL05B104KO5NNNC "
+		(property "PN" "187-CL05B104KO5NNNC"
 			(at 175.26 69.85 0)
 			(effects
@@
 			)
 		)
-		(property "PN" " 603-ANT8010LL05R1516 "
+		(property "PN" "603-ANT8010LL05R1516"
 			(at 181.61 99.06 0)
 			(effects
@@
 			)
 		)
-		(property "PN" " 187-CL05B104KO5NNNC "
+		(property "PN" "187-CL05B104KO5NNNC"
 			(at 140.97 69.85 0)
 			(effects
@@
 			)
 		)
-		(property "PN" " 187-CL05B104KO5NNNC "
+		(property "PN" "187-CL05B104KO5NNNC"
 			(at 116.84 69.85 0)
 			(effects
