File: gnss.kicad_sch (KiCad schematic)
At the start: 15 parts, among them U13 LG77L

Commit message: Changed GNSS antenna to a standard U.FL connector
Parts:
- removed AE1: ANT8010LL05R1516A, parts:ANT8010LL05R1516A, symbol Device:Antenna_Chip
- added J4: Conn_Coaxial, parts:Connector_ufl_1909763-1, symbol Connector:Conn_Coaxial
Connections:
- net GND: now also J4.2 (Ext)
- net at C20.1, R17.2: now also J4.1 (In)
- no-connect marks 4 -> 3
Changed lines of the file:
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@@
-	)
-	(no_connect
-		(at 184.15 101.6)
 	)
 	(no_connect
@@
 	(wire
 		(pts
+			(xy 186.69 107.95) (xy 186.69 113.03)
+		)
+		(stroke
+			(width 0)
+			(type default)
+		)
+	)
+	(wire
+		(pts
 			(xy 175.26 74.93) (xy 186.69 74.93)
 		)
@@
 	(wire
 		(pts
-			(xy 175.26 102.87) (xy 179.07 102.87)
+			(xy 175.26 102.87) (xy 181.61 102.87)
 		)
 		(stroke
@@
 	(wire
 		(pts
+			(xy 186.69 113.03) (xy 175.26 113.03)
+		)
+		(stroke
+			(width 0)
+			(type default)
+		)
+	)
+	(wire
+		(pts
 			(xy 154.94 120.65) (xy 165.1 120.65)
 		)
@@
 		(pts
 			(xy 186.69 74.93) (xy 186.69 73.66)
-		)
-		(stroke
-			(width 0)
-			(type default)
-		)
-	)
-	(wire
-		(pts
-			(xy 179.07 102.87) (xy 179.07 101.6)
 		)
 		(stroke
@@
 	)
 	(symbol
-		(lib_id "Device:Antenna_Chip")
-		(at 181.61 99.06 0)
+		(lib_id "Connector:Conn_Coaxial")
+		(at 186.69 102.87 0)
 		(unit 1)
 		(exclude_from_sim no)
@@
 		(on_board yes)
 		(dnp no)
-		(property "Reference" "AE1"
-			(at 181.356 95.504 0)
-			(effects
-				(font
-					(size 1.27 1.27)
-				)
-				(justify right)
-			)
-		)
-		(property "Value" "ANT8010LL05R1516A"
-			(at 181.356 92.964 0)
-			(effects
-				(font
-					(size 1.27 1.27)
-				)
-				(justify right)
-			)
-		)
-		(property "Footprint" "parts:ANT8010LL05R1516A"
-			(at 179.07 94.615 0)
+		(fields_autoplaced yes)
+		(property "Reference" "J4"
+			(at 190.5 101.8931 0)
+			(effects
+				(font
+					(size 1.27 1.27)
+				)
+				(justify left)
+			)
+		)
+		(property "Value" "Conn_Coaxial"
+			(at 190.5 104.4331 0)
+			(effects
+				(font
+					(size 1.27 1.27)
+				)
+				(justify left)
+			)
+		)
+		(property "Footprint" "parts:Connector_ufl_1909763-1"
+			(at 186.69 102.87 0)
 			(effects
 				(font
@@
 		)
 		(property "Datasheet" "~"
-			(at 179.07 94.615 0)
-			(effects
-				(font
-					(size 1.27 1.27)
-				)
-				(hide yes)
-			)
-		)
-		(property "Description" "Ceramic chip antenna with pin for PCB trace"
-			(at 181.61 99.06 0)
-			(effects
-				(font
-					(size 1.27 1.27)
-				)
-				(hide yes)
-			)
-		)
-		(property "LCSC" "C6740797"
-			(at 181.61 99.06 0)
-			(effects
-				(font
-					(size 1.27 1.27)
-				)
-				(hide yes)
-			)
-		)
-		(property "MPN" "ANT8010LL05R1516A"
-			(at 181.61 99.06 0)
-			(effects
-				(font
-					(size 1.27 1.27)
-				)
-				(hide yes)
-			)
-		)
-		(property "PN" "603-ANT8010LL05R1516"
-			(at 181.61 99.06 0)
-			(effects
-				(font
-					(size 1.27 1.27)
-				)
-				(hide yes)
-			)
+			(at 186.69 102.87 0)
+			(effects
+				(font
+					(size 1.27 1.27)
+				)
+				(hide yes)
+			)
+		)
+		(property "Description" "coaxial connector (BNC, SMA, SMB, SMC, Cinch/RCA, LEMO, ...)"
+			(at 186.69 102.87 0)
+			(effects
+				(font
+					(size 1.27 1.27)
+				)
+				(hide yes)
+			)
+		)
+		(property "LCSC" "C392444"
+			(at 186.69 102.87 0)
+			(effects
+				(font
+					(size 1.27 1.27)
+				)
+				(hide yes)
+			)
+		)
+		(property "MPN" "1909763-1"
+			(at 186.69 102.87 0)
+			(effects
+				(font
+					(size 1.27 1.27)
+				)
+				(hide yes)
+			)
+		)
+		(property "PN" "571-1909763-1"
+			(at 186.69 102.87 0)
+			(effects
+				(font
+					(size 1.27 1.27)
+				)
+				(hide yes)
+			)
+		)
+		(pin "2"
 		)
 		(pin "1"
-		)
-		(pin "2"
 		)
 		(instances
 			(project "linht-hw"
 				(path "/73efc1fc-21f6-4aef-9f73-508fe18fa32e/0b7c638a-0bf4-4df2-9e8c-e9dd4f727b29"
-					(reference "AE1")
+					(reference "J4")
 					(unit 1)
 				)
