File: gnss.kicad_sch (KiCad schematic)
At the start: 15 parts, among them J4 Conn_Coaxial, U13 LG77L

Commit message: minor tweaks to the Rev C
- KiCAD version update to 10.0.4
- added some more GND vias
- GNSS antenna connector placement change
- NOTE: one +5V track is left unconnected
Other:
- title: GNSS Module -> LinHT - Linux-based SDR handheld transceiver
